Commit message: Added more robots, changed ros2_control xacro

File: kuka_agilus_support/urdf/kr6_r700_sixx.urdf.xacro (robot description, xacro)
@@ -5,4 +5,22 @@
   <!-- Read additional arguments  -->
   <xacro:arg name="use_fake_hardware" default="false" />
-  <xacro:kuka_kr6_r700_sixx_robot prefix=""  use_fake_hardware="$(arg use_fake_hardware)"/>
+  <xacro:arg name="rsi_config_file" default="rsi_config.yaml" />
+  <xacro:arg name="namespace" default="" />
+  <!-- Turn the rsi config file argument into a property, for comparison-->
+  <xacro:property name="default_rsi_config_file" value="rsi_config.yaml"/>
+  <xacro:property name="current_rsi_config_file" value="$(arg rsi_config_file)"/>
+  <!-- Read parameters from rsi_config  -->
+  <xacro:property name="rsi_config" value="$(arg rsi_config_file)" />
+  <xacro:if value="${current_rsi_config_file == default_rsi_config_file}">
+      <xacro:property name="rsi_config_dict" value="${xacro.load_yaml(rsi_config)}"/>
+  </xacro:if>
+  <xacro:unless value="${current_rsi_config_file == default_rsi_config_file}">
+      <xacro:property name="rsi_config_dict" value="${xacro.load_yaml(rsi_config)}"/>
+  </xacro:unless>
+  <xacro:property name="client_ip" value="${rsi_config_dict['client_ip']}"/>
+  <xacro:property name="client_port" value="${rsi_config_dict['client_port']}" />
+  <xacro:kuka_kr6_r700_sixx_robot prefix="$(arg namespace)"
+                                  client_ip="${client_ip}"
+                                  client_port="${client_port}"
+                                  use_fake_hardware="$(arg use_fake_hardware)"/>
 </robot>

File: kuka_agilus_support/urdf/kr6_r700_sixx_macro.xacro (robot description, xacro)
@@ -5,9 +5,11 @@
   <xacro:include filename="$(find kuka_agilus_support)/urdf/kr_agilus_ros2_control.xacro" />
   <xacro:include filename="$(find kuka_agilus_support)/urdf/kr_agilus_transmission.xacro" />
-  <xacro:macro name="kuka_kr6_r700_sixx_robot" params="prefix use_fake_hardware">
+  <xacro:macro name="kuka_kr6_r700_sixx_robot" params="prefix client_ip client_port use_fake_hardware">
     <!-- ros2 control instance -->
     <xacro:kuka_agilus_ros2_control
     name="kr6_r700_sixx"
     prefix="${prefix}"
+    client_ip="${client_ip}"
+    client_port="${client_port}"
     use_fake_hardware="${use_fake_hardware}" />
     <link name="${prefix}base_link"/>

File: kuka_agilus_support/urdf/kr_agilus_ros2_control.xacro (robot description, xacro)
@@ -1,5 +1,5 @@
 <?xml version="1.0" encoding="UTF-8"?>
 <robot xmlns:xacro="http://www.ros.org/wiki/xacro">
-  <xacro:macro name="kuka_agilus_ros2_control" params="name prefix use_fake_hardware:=false">
+  <xacro:macro name="kuka_agilus_ros2_control" params="name prefix client_ip client_port use_fake_hardware:=false">
     <ros2_control name="${name}" type="system">
       <hardware>
@@ -11,8 +11,8 @@
         <xacro:unless value="${use_fake_hardware}">
           <!-- Read parameters from rsi_config  -->
-          <xacro:property name="rsi_config" value="$(find kuka_kss_rsi_driver)/config/driver_config.yaml" />
-          <xacro:property name="rsi_config_dict" value="${xacro.load_yaml(rsi_config)}"/>
+          <!-- <xacro:property name="rsi_config" value="$(find kuka_kss_rsi_driver)/config/driver_config.yaml" /> -->
+          <!-- <xacro:property name="rsi_config_dict" value="${xacro.load_yaml(rsi_config)}"/>
           <xacro:property name="client_ip" value="${rsi_config_dict['client_ip']}" />
-          <xacro:property name="client_port" value="${rsi_config_dict['client_port']}" />
+          <xacro:property name="client_port" value="${rsi_config_dict['client_port']}" /> -->
           <plugin>kuka_kss_rsi_driver::KukaRSIHardwareInterface</plugin>
           <param name="client_ip">${client_ip}</param>

File: kuka_quantec_support/urdf/kr_quantec_ros2_control.xacro (robot description, xacro)
@@ -1,5 +1,5 @@
 <?xml version="1.0" encoding="UTF-8"?>
 <robot xmlns:xacro="http://www.ros.org/wiki/xacro">
-  <xacro:macro name="kuka_quantec_ros2_control" params="name prefix use_fake_hardware:=false">
+  <xacro:macro name="kuka_quantec_ros2_control" params="name prefix client_ip client_port use_fake_hardware:=false">
     <ros2_control name="${name}" type="system">
       <hardware>
@@ -11,8 +11,8 @@
         <xacro:unless value="${use_fake_hardware}">
           <!-- Read parameters from rsi_config  -->
-          <xacro:property name="rsi_config" value="$(find kuka_kss_rsi_driver)/config/driver_config.yaml" />
+          <!-- <xacro:property name="rsi_config" value="$(find kuka_kss_rsi_driver)/config/driver_config.yaml" />
           <xacro:property name="rsi_config_dict" value="${xacro.load_yaml(rsi_config)}"/>
           <xacro:property name="client_ip" value="${rsi_config_dict['client_ip']}" />
-          <xacro:property name="client_port" value="${rsi_config_dict['client_port']}" />
+          <xacro:property name="client_port" value="${rsi_config_dict['client_port']}" /> -->
           <plugin>kuka_kss_rsi_driver::KukaRSIHardwareInterface</plugin>
           <param name="client_ip">${client_ip}</param>

Commit message: fixed xacro stuff

File: kuka_agilus_support/urdf/kr6_r700_sixx.urdf.xacro (robot description, xacro)
@@ -5,15 +5,16 @@
   <!-- Read additional arguments  -->
   <xacro:arg name="use_fake_hardware" default="false" />
-  <xacro:arg name="rsi_config_file" default="rsi_config.yaml" />
+  <xacro:arg name="rsi_config_file" default="driver_config.yaml" />
   <xacro:arg name="namespace" default="" />
   <!-- Turn the rsi config file argument into a property, for comparison-->
-  <xacro:property name="default_rsi_config_file" value="rsi_config.yaml"/>
+  <xacro:property name="default_rsi_config_file" value="driver_config.yaml"/>
   <xacro:property name="current_rsi_config_file" value="$(arg rsi_config_file)"/>
   <!-- Read parameters from rsi_config  -->
-  <xacro:property name="rsi_config" value="$(arg rsi_config_file)" />
   <xacro:if value="${current_rsi_config_file == default_rsi_config_file}">
+      <xacro:property name="rsi_config" value="$(find kuka_kss_rsi_driver)/config/$(arg rsi_config_file)"/>
       <xacro:property name="rsi_config_dict" value="${xacro.load_yaml(rsi_config)}"/>
   </xacro:if>
   <xacro:unless value="${current_rsi_config_file == default_rsi_config_file}">
+      <xacro:property name="rsi_config" value="$(arg rsi_config_file)" />
       <xacro:property name="rsi_config_dict" value="${xacro.load_yaml(rsi_config)}"/>
   </xacro:unless>

File: kuka_agilus_support/urdf/kr_agilus_ros2_control.xacro (robot description, xacro)
@@ -23,5 +23,5 @@
         <command_interface name="position"/>
       <state_interface name="position">
-        <param name="initial_value">-1.5708</param>
+        <param name="initial_value">0</param>
       </state_interface>
       </joint>
@@ -29,5 +29,5 @@
         <command_interface name="position"/>
       <state_interface name="position">
-        <param name="initial_value">1.13</param>
+        <param name="initial_value">0</param>
       </state_interface>
       </joint>
@@ -35,5 +35,5 @@
         <command_interface name="position"/>
       <state_interface name="position">
-        <param name="initial_value">-2.4</param>
+        <param name="initial_value">0.0</param>
       </state_interface>
       </joint>
