Commit message: Made kr8 description match the naming scheme of other robots

File: kuka_agilus_support/urdf/kr8_r1640-2_macro.xacro (robot description, xacro)
@@ -17,5 +17,5 @@
         <origin xyz="0 0 0" rpy="0 0 0" />
         <geometry>
-          <mesh filename="package://kuka_agilus_support/meshes/kr8_r1640-2/meshes/base_link.STL" />
+          <mesh filename="package://kuka_agilus_support/meshes/kr8_r1640-2/visual/base_link.STL" />
         </geometry>
         <xacro:material_kuka_pedestal />
@@ -24,5 +24,5 @@
         <origin xyz="0 0 0" rpy="0 0 0" />
         <geometry>
-          <mesh filename="package://kuka_agilus_support/meshes/kr8_r1640-2/meshes/base_link.STL" />
+          <mesh filename="package://kuka_agilus_support/meshes/kr8_r1640-2/visual/base_link.STL" />
         </geometry>
       </collision>
@@ -46,12 +46,12 @@
         <origin xyz="0 0 0" rpy="0 0 0" />
         <geometry>
-          <mesh filename="package://kuka_agilus_support/meshes/kr8_r1640-2/meshes/lr_link1.STL" />
-        </geometry>
-        <xacro:material_kuka_orange />
-      </visual>
-      <collision>
-        <origin xyz="0 0 0" rpy="0 0 0" />
-        <geometry>
-          <mesh filename="package://kuka_agilus_support/meshes/kr8_r1640-2/meshes/lr_link1.STL" />
+          <mesh filename="package://kuka_agilus_support/meshes/kr8_r1640-2/visual/link_1.STL" />
+        </geometry>
+        <xacro:material_kuka_orange />
+      </visual>
+      <collision>
+        <origin xyz="0 0 0" rpy="0 0 0" />
+        <geometry>
+          <mesh filename="package://kuka_agilus_support/meshes/kr8_r1640-2/visual/link_1.STL" />
         </geometry>
       </collision>
@@ -75,12 +75,12 @@
         <origin xyz="0 0 0" rpy="0 0 0" />
         <geometry>
-          <mesh filename="package://kuka_agilus_support/meshes/kr8_r1640-2/meshes/lr_link2.STL" />
-        </geometry>
-        <xacro:material_kuka_orange />
-      </visual>
-      <collision>
-        <origin xyz="0 0 0" rpy="0 0 0" />
-        <geometry>
-          <mesh filename="package://kuka_agilus_support/meshes/kr8_r1640-2/meshes/lr_link2.STL" />
+          <mesh filename="package://kuka_agilus_support/meshes/kr8_r1640-2/visual/link_2.STL" />
+        </geometry>
+        <xacro:material_kuka_orange />
+      </visual>
+      <collision>
+        <origin xyz="0 0 0" rpy="0 0 0" />
+        <geometry>
+          <mesh filename="package://kuka_agilus_support/meshes/kr8_r1640-2/visual/link_2.STL" />
         </geometry>
       </collision>
@@ -104,12 +104,12 @@
         <origin xyz="0 0 0" rpy="0 0 0" />
         <geometry>
-          <mesh filename="package://kuka_agilus_support/meshes/kr8_r1640-2/meshes/lr_link3.STL" />
-        </geometry>
-        <xacro:material_kuka_orange />
-      </visual>
-      <collision>
-        <origin xyz="0 0 0" rpy="0 0 0" />
-        <geometry>
-          <mesh filename="package://kuka_agilus_support/meshes/kr8_r1640-2/meshes/lr_link3.STL" />
+          <mesh filename="package://kuka_agilus_support/meshes/kr8_r1640-2/visual/link_3.STL" />
+        </geometry>
+        <xacro:material_kuka_orange />
+      </visual>
+      <collision>
+        <origin xyz="0 0 0" rpy="0 0 0" />
+        <geometry>
+          <mesh filename="package://kuka_agilus_support/meshes/kr8_r1640-2/visual/link_3.STL" />
         </geometry>
       </collision>
@@ -133,12 +133,12 @@
         <origin xyz="0 0 0" rpy="0 0 0" />
         <geometry>
-          <mesh filename="package://kuka_agilus_support/meshes/kr8_r1640-2/meshes/lr_link4.STL" />
-        </geometry>
-        <xacro:material_kuka_orange />
-      </visual>
-      <collision>
-        <origin xyz="0 0 0" rpy="0 0 0" />
-        <geometry>
-          <mesh filename="package://kuka_agilus_support/meshes/kr8_r1640-2/meshes/lr_link4.STL" />
+          <mesh filename="package://kuka_agilus_support/meshes/kr8_r1640-2/visual/link_4.STL" />
+        </geometry>
+        <xacro:material_kuka_orange />
+      </visual>
+      <collision>
+        <origin xyz="0 0 0" rpy="0 0 0" />
+        <geometry>
+          <mesh filename="package://kuka_agilus_support/meshes/kr8_r1640-2/visual/link_4.STL" />
         </geometry>
       </collision>
@@ -162,12 +162,12 @@
         <origin xyz="0 0 0" rpy="0 0 0" />
         <geometry>
-          <mesh filename="package://kuka_agilus_support/meshes/kr8_r1640-2/meshes/lr_link5.STL" />
-        </geometry>
-        <xacro:material_kuka_orange />
-      </visual>
-      <collision>
-        <origin xyz="0 0 0" rpy="0 0 0" />
-        <geometry>
-          <mesh filename="package://kuka_agilus_support/meshes/kr8_r1640-2/meshes/lr_link5.STL" />
+          <mesh filename="package://kuka_agilus_support/meshes/kr8_r1640-2/visual/link_5.STL" />
+        </geometry>
+        <xacro:material_kuka_orange />
+      </visual>
+      <collision>
+        <origin xyz="0 0 0" rpy="0 0 0" />
+        <geometry>
+          <mesh filename="package://kuka_agilus_support/meshes/kr8_r1640-2/visual/link_5.STL" />
         </geometry>
       </collision>
@@ -191,5 +191,5 @@
         <origin xyz="0 0 0" rpy="3.1415926539 0 0" />
         <geometry>
-          <mesh filename="package://kuka_agilus_support/meshes/kr8_r1640-2/meshes/lr_link6.STL" />
+          <mesh filename="package://kuka_agilus_support/meshes/kr8_r1640-2/visual/link_6.STL" />
         </geometry>
         <xacro:material_kuka_pedestal />
@@ -198,5 +198,5 @@
         <origin xyz="0 0 0" rpy="3.1415926539 0 0" />
         <geometry>
-          <mesh filename="package://kuka_agilus_support/meshes/kr8_r1640-2/meshes/lr_link6.STL" />
+          <mesh filename="package://kuka_agilus_support/meshes/kr8_r1640-2/visual/link_6.STL" />
         </geometry>
       </collision>

File: kuka_agilus_support/urdf/kr_agilus_ros2_control.xacro (robot description, xacro)
@@ -23,5 +23,5 @@
         <command_interface name="position"/>
       <state_interface name="position">
-        <param name="initial_value">0.0</param>
+        <param name="initial_value">-1.5708</param>
       </state_interface>
       </joint>
@@ -29,5 +29,5 @@
         <command_interface name="position"/>
       <state_interface name="position">
-        <param name="initial_value">0.0</param>
+        <param name="initial_value">1.13</param>
       </state_interface>
       </joint>
@@ -35,5 +35,5 @@
         <command_interface name="position"/>
       <state_interface name="position">
-        <param name="initial_value">0.0</param>
+        <param name="initial_value">-2.4</param>
       </state_interface>
       </joint>

Commit message: fixing flange orientation

File: kuka_agilus_support/urdf/kr8_r1640-2_macro.xacro (robot description, xacro)
@@ -288,5 +288,5 @@
       <parent link="${prefix}link_6"/>
       <child link="${prefix}flange"/>
-      <origin xyz="0 0 0" rpy="0 0 0"/>
+      <origin xyz="0 0 0" rpy="0 1.5708 0"/>
     </joint>
     <!-- ROS base_link to KUKA $ROBROOT coordinate system transform -->
