Commit message: Fixed URDF for kr8_r1640_2
Also made xacro usable without RSI inputs

File: kuka_agilus_support/urdf/kr8_r1640-2.urdf.xacro (robot description, xacro)
@@ -12,19 +12,27 @@
 <xacro:arg name="rsi_config_file" default="rsi_config.yaml" />
 <xacro:arg name="namespace" default="" />
-<!-- Turn the rsi config file argument into a property, for comparison-->
-<xacro:property name="default_rsi_config_file" value="rsi_config.yaml"/>
-<xacro:property name="current_rsi_config_file" value="$(arg rsi_config_file)"/>
-<!-- Read parameters from rsi_config  -->
-<xacro:property name="rsi_config" value="$(arg rsi_config_file)" />
-<xacro:if value="${current_rsi_config_file == default_rsi_config_file}">
-    <xacro:property name="rsi_config_dict" value="${xacro.load_yaml(rsi_config)}"/>
+<xacro:property name="use_fake_hardware_prop" value="$(arg use_fake_hardware)"/>
+<xacro:property name="false_prop" value="false"/>
+<xacro:unless value="${use_fake_hardware_prop == false_prop}">
+    <!-- Turn the rsi config file argument into a property, for comparison-->
+    <xacro:property name="default_rsi_config_file" value="rsi_config.yaml"/>
+    <xacro:property name="current_rsi_config_file" value="$(arg rsi_config_file)"/>
+    <!-- Read parameters from rsi_config  -->
+    <xacro:property name="rsi_config" value="$(arg rsi_config_file)" />
+    <xacro:if value="${current_rsi_config_file == default_rsi_config_file}">
+        <xacro:property name="rsi_config_dict" value="${xacro.load_yaml(rsi_config)}"/>
+    </xacro:if>
+    <xacro:unless value="${current_rsi_config_file == default_rsi_config_file}">
+        <xacro:property name="rsi_config_dict" value="${xacro.load_yaml(rsi_config)}"/>
+    </xacro:unless>
+    <xacro:property name="client_ip" value="${rsi_config_dict['client_ip']}"/>
+    <xacro:property name="client_port" value="${rsi_config_dict['client_port']}" />
+</xacro:unless>
+<xacro:if value="${use_fake_hardware_prop == false_prop}">
+    <xacro:property name="client_ip" value="0.0.0.0"/>
+    <xacro:property name="client_port" value="0" />
 </xacro:if>
-<xacro:unless value="${current_rsi_config_file == default_rsi_config_file}">
-    <xacro:property name="rsi_config_dict" value="${xacro.load_yaml(rsi_config)}"/>
-</xacro:unless>
-<xacro:property name="client_ip" value="${rsi_config_dict['client_ip']}"/>
-<xacro:property name="client_port" value="${rsi_config_dict['client_port']}" />
 <!-- Read additional arguments  -->
-<xacro:arg name="use_fake_hardware" default="false" />
+<!-- <xacro:arg name="use_fake_hardware" default="false" /> -->
 <xacro:kr8_r1640-2_robot prefix="$(arg namespace)"
                   client_ip="${client_ip}"

File: kuka_agilus_support/urdf/kr8_r1640-2_macro.xacro (robot description, xacro)
@@ -44,5 +44,5 @@
     <link name="${prefix}link_1">
       <visual>
-        <origin xyz="0 0 0" rpy="0 0 0" />
+        <origin xyz="0 0 -.21195" rpy="0 0 0" />
         <geometry>
           <mesh filename="package://kuka_agilus_support/meshes/kr8_r1640-2/visual/link_1.STL" />
@@ -51,5 +51,5 @@
       </visual>
       <collision>
-        <origin xyz="0 0 0" rpy="0 0 0" />
+        <origin xyz="0 0 -0.21195" rpy="0 0 0" />
         <geometry>
           <mesh filename="package://kuka_agilus_support/meshes/kr8_r1640-2/visual/link_1.STL" />
@@ -73,5 +73,5 @@
     <link name="${prefix}link_2">
       <visual>
-        <origin xyz="0 0 0" rpy="0 0 0" />
+        <origin xyz="0 -0.051664 0" rpy="0 0 0" />
         <geometry>
           <mesh filename="package://kuka_agilus_support/meshes/kr8_r1640-2/visual/link_2.STL" />
@@ -80,5 +80,5 @@
       </visual>
       <collision>
-        <origin xyz="0 0 0" rpy="0 0 0" />
+        <origin xyz="0 -0.051664 0" rpy="0 0 0" />
         <geometry>
           <mesh filename="package://kuka_agilus_support/meshes/kr8_r1640-2/visual/link_2.STL" />
@@ -102,5 +102,5 @@
     <link name="${prefix}link_3">
       <visual>
-        <origin xyz="0 0 0" rpy="0 0 0" />
+        <origin xyz="0 -0.051664 0" rpy="0 0 0" />
         <geometry>
           <mesh filename="package://kuka_agilus_support/meshes/kr8_r1640-2/visual/link_3.STL" />
@@ -109,5 +109,5 @@
       </visual>
       <collision>
-        <origin xyz="0 0 0" rpy="0 0 0" />
+        <origin xyz="0 -0.051664 0" rpy="0 0 0" />
         <geometry>
           <mesh filename="package://kuka_agilus_support/meshes/kr8_r1640-2/visual/link_3.STL" />
@@ -131,5 +131,5 @@
     <link name="${prefix}link_4">
       <visual>
-        <origin xyz="0 0 0" rpy="0 0 0" />
+        <origin xyz="-0.3175 0 0" rpy="0 0 0" />
         <geometry>
           <mesh filename="package://kuka_agilus_support/meshes/kr8_r1640-2/visual/link_4.STL" />
@@ -138,5 +138,5 @@
       </visual>
       <collision>
-        <origin xyz="0 0 0" rpy="0 0 0" />
+        <origin xyz="-0.3175 0 0" rpy="0 0 0" />
         <geometry>
           <mesh filename="package://kuka_agilus_support/meshes/kr8_r1640-2/visual/link_4.STL" />
@@ -160,5 +160,5 @@
     <link name="${prefix}link_5">
       <visual>
-        <origin xyz="0 0 0" rpy="0 0 0" />
+        <origin xyz="0 -0.0015 0" rpy="0 0 0" />
         <geometry>
           <mesh filename="package://kuka_agilus_support/meshes/kr8_r1640-2/visual/link_5.STL" />
@@ -167,5 +167,5 @@
       </visual>
       <collision>
-        <origin xyz="0 0 0" rpy="0 0 0" />
+        <origin xyz="0 -0.0015 0" rpy="0 0 0" />
         <geometry>
           <mesh filename="package://kuka_agilus_support/meshes/kr8_r1640-2/visual/link_5.STL" />
@@ -189,5 +189,5 @@
     <link name="${prefix}link_6">
       <visual>
-        <origin xyz="0 0 0" rpy="3.1415926539 0 0" />
+        <origin xyz="-0.0175 0 0" rpy="3.1415926539 0 0" />
         <geometry>
           <mesh filename="package://kuka_agilus_support/meshes/kr8_r1640-2/visual/link_6.STL" />
@@ -196,5 +196,5 @@
       </visual>
       <collision>
-        <origin xyz="0 0 0" rpy="3.1415926539 0 0" />
+        <origin xyz="-0.0175 0 0" rpy="3.1415926539 0 0" />
         <geometry>
           <mesh filename="package://kuka_agilus_support/meshes/kr8_r1640-2/visual/link_6.STL" />
@@ -220,6 +220,6 @@
     <joint name="${prefix}joint_a1" type="revolute">
       <origin
-        xyz="0 0 0.21195"
-        rpy="0 0 0.013412" />
+        xyz="0 0 0.425"
+        rpy="0 0 0.0" />
       <parent link="${prefix}base_link"/>
       <child link="${prefix}link_1"/>
@@ -231,6 +231,8 @@
     </joint>
     <joint name="${prefix}joint_a2" type="revolute">
-      <origin xyz="0.17 -0.051664 0.21305"
-        rpy="0 1.5708 0" />
+      <!-- <origin xyz="0.17 -0.051664 0.21305"
+        rpy="0 1.5708 0" /> -->
+      <origin xyz="0.17 0.0 0.0"
+        rpy="0 1.57079632679 0" />
       <parent link="${prefix}link_1"/>
       <child link="${prefix}link_2"/>
@@ -243,5 +245,5 @@
     <joint name="${prefix}joint_a3" type="revolute">
       <origin xyz="0 0 0.81"
-        rpy="0 -1.5708 0" />
+        rpy="0 -1.57079632679 0" />
       <parent link="${prefix}link_2"/>
       <child link="${prefix}link_3"/>
@@ -253,6 +255,6 @@
     </joint>
     <joint name="${prefix}joint_a4" type="revolute">
-      <origin xyz="0.34178 0.051664 0.02"
-        rpy="-0.0066973 0 0" />
+      <origin xyz="0.66 0.0 0.02"
+        rpy="0 0 0" />
       <parent link="${prefix}link_3"/>
       <child link="${prefix}link_4"/>
@@ -264,6 +266,6 @@
     </joint>
     <joint name="${prefix}joint_a5" type="revolute">
-      <origin xyz="0.31822 0 0"
-        rpy="0 0.064576 0" />
+      <origin xyz="0.0 0 0"
+        rpy="0 0.0 0" />
       <parent link="${prefix}link_4"/>
       <child link="${prefix}link_5"/>
@@ -275,5 +277,5 @@
     </joint>
     <joint name="${prefix}joint_a6" type="revolute">
-      <origin xyz="0.08224 0.001 0"
+      <origin xyz="0.1 0.0 0.0"
         rpy="0 0 0" />
       <parent link="${prefix}link_5"/>
