Commit message: Fixed naming, added simpler collision meshes to kr8_r1640

File: kuka_agilus_support/urdf/kr8_r1640_2.urdf.xacro (robot description, xacro)
@@ -1,6 +1,6 @@
 <?xml version="1.0"?>
-<robot xmlns:xacro="http://www.ros.org/wiki/xacro" name="kr8_r1640-2">
+<robot xmlns:xacro="http://www.ros.org/wiki/xacro" name="kr8_r1640_2">
 <!-- Import urdf file  -->
-<xacro:include filename="$(find kuka_agilus_support)/urdf/kr8_r1640-2_macro.xacro"/>
+<xacro:include filename="$(find kuka_agilus_support)/urdf/kr8_r1640_2_macro.xacro"/>
 <!-- Read parameters from rsi_config  -->
 <!-- <xacro:property name="rsi_config" value="$(find kuka_rsi_hw_interface)/config/rsi_config.yaml" />

File: kuka_agilus_support/urdf/kr8_r1640_2_macro.xacro (robot description, xacro)
@@ -5,8 +5,8 @@
   <xacro:include filename="$(find kuka_agilus_support)/urdf/kr_agilus_ros2_control.xacro" />
   <xacro:include filename="$(find kuka_agilus_support)/urdf/kr_agilus_transmission.xacro" />
-  <xacro:macro name="kr8_r1640-2_robot" params="prefix client_ip client_port use_fake_hardware">
+  <xacro:macro name="kr8_r1640_2_robot" params="prefix client_ip client_port use_fake_hardware">
     <!-- ros2 control instance -->
     <xacro:kuka_agilus_ros2_control
-    name="kr8_r1640-2"
+    name="kr8_r1640_2"
     prefix="${prefix}"
     client_ip="${client_ip}"
@@ -17,5 +17,5 @@
         <origin xyz="0 0 0" rpy="0 0 0" />
         <geometry>
-          <mesh filename="package://kuka_agilus_support/meshes/kr8_r1640-2/visual/base_link.STL" />
+          <mesh filename="package://kuka_agilus_support/meshes/kr8_r1640_2/visual/base_link.STL" />
         </geometry>
         <xacro:material_kuka_pedestal />
@@ -24,5 +24,5 @@
         <origin xyz="0 0 0" rpy="0 0 0" />
         <geometry>
-          <mesh filename="package://kuka_agilus_support/meshes/kr8_r1640-2/visual/base_link.STL" />
+          <mesh filename="package://kuka_agilus_support/meshes/kr8_r1640_2/collision/base_link.stl" />
         </geometry>
       </collision>
@@ -46,5 +46,5 @@
         <origin xyz="0 0 -.21195" rpy="0 0 0" />
         <geometry>
-          <mesh filename="package://kuka_agilus_support/meshes/kr8_r1640-2/visual/link_1.STL" />
+          <mesh filename="package://kuka_agilus_support/meshes/kr8_r1640_2/visual/link_1.STL" />
         </geometry>
         <xacro:material_kuka_orange />
@@ -53,5 +53,5 @@
         <origin xyz="0 0 -0.21195" rpy="0 0 0" />
         <geometry>
-          <mesh filename="package://kuka_agilus_support/meshes/kr8_r1640-2/visual/link_1.STL" />
+          <mesh filename="package://kuka_agilus_support/meshes/kr8_r1640_2/collision/link_1.stl" />
         </geometry>
       </collision>
@@ -75,5 +75,5 @@
         <origin xyz="0 -0.051664 0" rpy="0 0 0" />
         <geometry>
-          <mesh filename="package://kuka_agilus_support/meshes/kr8_r1640-2/visual/link_2.STL" />
+          <mesh filename="package://kuka_agilus_support/meshes/kr8_r1640_2/visual/link_2.STL" />
         </geometry>
         <xacro:material_kuka_orange />
@@ -82,5 +82,5 @@
         <origin xyz="0 -0.051664 0" rpy="0 0 0" />
         <geometry>
-          <mesh filename="package://kuka_agilus_support/meshes/kr8_r1640-2/visual/link_2.STL" />
+          <mesh filename="package://kuka_agilus_support/meshes/kr8_r1640_2/collision/link_2.stl" />
         </geometry>
       </collision>
@@ -104,5 +104,5 @@
         <origin xyz="0 -0.051664 0" rpy="0 0 0" />
         <geometry>
-          <mesh filename="package://kuka_agilus_support/meshes/kr8_r1640-2/visual/link_3.STL" />
+          <mesh filename="package://kuka_agilus_support/meshes/kr8_r1640_2/visual/link_3.STL" />
         </geometry>
         <xacro:material_kuka_orange />
@@ -111,5 +111,5 @@
         <origin xyz="0 -0.051664 0" rpy="0 0 0" />
         <geometry>
-          <mesh filename="package://kuka_agilus_support/meshes/kr8_r1640-2/visual/link_3.STL" />
+          <mesh filename="package://kuka_agilus_support/meshes/kr8_r1640_2/collision/link_3.stl" />
         </geometry>
       </collision>
@@ -133,5 +133,5 @@
         <origin xyz="-0.3175 0 0" rpy="0 0 0" />
         <geometry>
-          <mesh filename="package://kuka_agilus_support/meshes/kr8_r1640-2/visual/link_4.STL" />
+          <mesh filename="package://kuka_agilus_support/meshes/kr8_r1640_2/visual/link_4.STL" />
         </geometry>
         <xacro:material_kuka_orange />
@@ -140,5 +140,5 @@
         <origin xyz="-0.3175 0 0" rpy="0 0 0" />
         <geometry>
-          <mesh filename="package://kuka_agilus_support/meshes/kr8_r1640-2/visual/link_4.STL" />
+          <mesh filename="package://kuka_agilus_support/meshes/kr8_r1640_2/collision/link_4.stl" />
         </geometry>
       </collision>
@@ -162,5 +162,5 @@
         <origin xyz="0 -0.0015 0" rpy="0 0 0" />
         <geometry>
-          <mesh filename="package://kuka_agilus_support/meshes/kr8_r1640-2/visual/link_5.STL" />
+          <mesh filename="package://kuka_agilus_support/meshes/kr8_r1640_2/visual/link_5.STL" />
         </geometry>
         <xacro:material_kuka_orange />
@@ -169,5 +169,5 @@
         <origin xyz="0 -0.0015 0" rpy="0 0 0" />
         <geometry>
-          <mesh filename="package://kuka_agilus_support/meshes/kr8_r1640-2/visual/link_5.STL" />
+          <mesh filename="package://kuka_agilus_support/meshes/kr8_r1640_2/collision/link_5.stl" />
         </geometry>
       </collision>
@@ -191,5 +191,5 @@
         <origin xyz="-0.0175 0 0" rpy="3.1415926539 0 0" />
         <geometry>
-          <mesh filename="package://kuka_agilus_support/meshes/kr8_r1640-2/visual/link_6.STL" />
+          <mesh filename="package://kuka_agilus_support/meshes/kr8_r1640_2/visual/link_6.STL" />
         </geometry>
         <xacro:material_kuka_pedestal />
@@ -198,5 +198,5 @@
         <origin xyz="-0.0175 0 0" rpy="3.1415926539 0 0" />
         <geometry>
-          <mesh filename="package://kuka_agilus_support/meshes/kr8_r1640-2/visual/link_6.STL" />
+          <mesh filename="package://kuka_agilus_support/meshes/kr8_r1640_2/collision/link_6.stl" />
         </geometry>
       </collision>
