Commit message: changed back the joint names

File: kuka_agilus_support/urdf/kr_agilus_ros2_control.xacro (robot description, xacro)
@@ -20,5 +20,5 @@
         </xacro:unless>
       </hardware>
-      <joint name="${prefix}joint_1">
+      <joint name="${prefix}joint_a1">
         <command_interface name="position"/>
       <state_interface name="position">
@@ -26,5 +26,5 @@
       </state_interface>
       </joint>
-      <joint name="${prefix}joint_2">
+      <joint name="${prefix}joint_a2">
         <command_interface name="position"/>
       <state_interface name="position">
@@ -32,5 +32,5 @@
       </state_interface>
       </joint>
-      <joint name="${prefix}joint_3">
+      <joint name="${prefix}joint_a3">
         <command_interface name="position"/>
       <state_interface name="position">
@@ -38,5 +38,5 @@
       </state_interface>
       </joint>
-      <joint name="${prefix}joint_4">
+      <joint name="${prefix}joint_a4">
         <command_interface name="position"/>
       <state_interface name="position">
@@ -44,5 +44,5 @@
       </state_interface>
       </joint>
-      <joint name="${prefix}joint_5">
+      <joint name="${prefix}joint_a5">
         <command_interface name="position"/>
       <state_interface name="position">
@@ -50,5 +50,5 @@
       </state_interface>
       </joint>
-      <joint name="${prefix}joint_6">
+      <joint name="${prefix}joint_a6">
         <command_interface name="position"/>
       <state_interface name="position">

File: kuka_quantec_support/urdf/kr_quantec_ros2_control.xacro (robot description, xacro)
@@ -20,5 +20,5 @@
         </xacro:unless>
       </hardware>
-      <joint name="${prefix}joint_1">
+      <joint name="${prefix}joint_a1">
         <command_interface name="position"/>
       <state_interface name="position">
@@ -26,5 +26,5 @@
       </state_interface>
       </joint>
-      <joint name="${prefix}joint_2">
+      <joint name="${prefix}joint_a2">
         <command_interface name="position"/>
       <state_interface name="position">
@@ -32,5 +32,5 @@
       </state_interface>
       </joint>
-      <joint name="${prefix}joint_3">
+      <joint name="${prefix}joint_a3">
         <command_interface name="position"/>
       <state_interface name="position">
@@ -38,5 +38,5 @@
       </state_interface>
       </joint>
-      <joint name="${prefix}joint_4">
+      <joint name="${prefix}joint_a4">
         <command_interface name="position"/>
       <state_interface name="position">
@@ -44,5 +44,5 @@
       </state_interface>
       </joint>
-      <joint name="${prefix}joint_5">
+      <joint name="${prefix}joint_a5">
         <command_interface name="position"/>
       <state_interface name="position">
@@ -50,5 +50,5 @@
       </state_interface>
       </joint>
-      <joint name="${prefix}joint_6">
+      <joint name="${prefix}joint_a6">
         <command_interface name="position"/>
       <state_interface name="position">

Commit message: wip

File: kuka_agilus_support/urdf/kr_agilus_ros2_control.xacro (robot description, xacro)
@@ -2,59 +2,4 @@
 <robot xmlns:xacro="http://www.ros.org/wiki/xacro">
   <xacro:macro name="kuka_agilus_ros2_control" params="name prefix client_ip client_port use_fake_hardware:=false">
-    <ros2_control name="${name}" type="system">
-      <hardware>
-        <xacro:if value="${use_fake_hardware}">
-          <plugin>mock_components/GenericSystem</plugin>
-          <param name="mock_sensor_commands">false</param>
-          <param name="state_following_offset">0.0</param>
-        </xacro:if>
-        <xacro:unless value="${use_fake_hardware}">
-          <!-- Read parameters from rsi_config  -->
-          <!-- <xacro:property name="rsi_config" value="$(find kuka_kss_rsi_driver)/config/driver_config.yaml" /> -->
-          <!-- <xacro:property name="rsi_config_dict" value="${xacro.load_yaml(rsi_config)}"/>
-          <xacro:property name="client_ip" value="${rsi_config_dict['client_ip']}" />
-          <xacro:property name="client_port" value="${rsi_config_dict['client_port']}" /> -->
-          <plugin>kuka_kss_rsi_driver::KukaRSIHardwareInterface</plugin>
-          <param name="client_ip">${client_ip}</param>
-          <param name="client_port">${client_port}</param>
-        </xacro:unless>
-      </hardware>
-      <joint name="${prefix}joint_a1">
-        <command_interface name="position"/>
-      <state_interface name="position">
-        <param name="initial_value">0</param>
-      </state_interface>
-      </joint>
-      <joint name="${prefix}joint_a2">
-        <command_interface name="position"/>
-      <state_interface name="position">
-        <param name="initial_value">0</param>
-      </state_interface>
-      </joint>
-      <joint name="${prefix}joint_a3">
-        <command_interface name="position"/>
-      <state_interface name="position">
-        <param name="initial_value">0.0</param>
-      </state_interface>
-      </joint>
-      <joint name="${prefix}joint_a4">
-        <command_interface name="position"/>
-      <state_interface name="position">
-        <param name="initial_value">0.0</param>
-      </state_interface>
-      </joint>
-      <joint name="${prefix}joint_a5">
-        <command_interface name="position"/>
-      <state_interface name="position">
-        <param name="initial_value">0.0</param>
-      </state_interface>
-      </joint>
-      <joint name="${prefix}joint_a6">
-        <command_interface name="position"/>
-      <state_interface name="position">
-        <param name="initial_value">0.0</param>
-      </state_interface>
-      </joint>
-    </ros2_control>
   </xacro:macro>
 </robot>

File: kuka_quantec_support/urdf/kr150_r3100-2_macro.xacro (robot description, xacro)
@@ -231,5 +231,5 @@
       <child link="${prefix}link_2"/>
       <axis xyz="0 1 0"/>
-      <limit effort="0" lower="${radians(-140)}" upper="${radians(-5)}" velocity="${radians(107)}"/>
+      <limit effort="0" lower="${radians(-140)}" upper="${radians(180)}" velocity="${radians(107)}"/>
     </joint>
     <joint name="${prefix}joint_a3" type="revolute">

File: kuka_quantec_support/urdf/kr_quantec_ros2_control.xacro (robot description, xacro)
@@ -2,59 +2,4 @@
 <robot xmlns:xacro="http://www.ros.org/wiki/xacro">
   <xacro:macro name="kuka_quantec_ros2_control" params="name prefix client_ip client_port use_fake_hardware:=false">
-    <ros2_control name="${name}" type="system">
-      <hardware>
-        <xacro:if value="${use_fake_hardware}">
-          <plugin>mock_components/GenericSystem</plugin>
-          <param name="mock_sensor_commands">false</param>
-          <param name="state_following_offset">0.0</param>
-        </xacro:if>
-        <xacro:unless value="${use_fake_hardware}">
-          <!-- Read parameters from rsi_config  -->
-          <!-- <xacro:property name="rsi_config" value="$(find kuka_kss_rsi_driver)/config/driver_config.yaml" />
-          <xacro:property name="rsi_config_dict" value="${xacro.load_yaml(rsi_config)}"/>
-          <xacro:property name="client_ip" value="${rsi_config_dict['client_ip']}" />
-          <xacro:property name="client_port" value="${rsi_config_dict['client_port']}" /> -->
-          <plugin>kuka_kss_rsi_driver::KukaRSIHardwareInterface</plugin>
-          <param name="client_ip">${client_ip}</param>
-          <param name="client_port">${client_port}</param>
-        </xacro:unless>
-      </hardware>
-      <joint name="${prefix}joint_a1">
-        <command_interface name="position"/>
-      <state_interface name="position">
-        <param name="initial_value">0.0</param>
-      </state_interface>
-      </joint>
-      <joint name="${prefix}joint_a2">
-        <command_interface name="position"/>
-      <state_interface name="position">
-        <param name="initial_value">-1.570796</param>
-      </state_interface>
-      </joint>
-      <joint name="${prefix}joint_a3">
-        <command_interface name="position"/>
-      <state_interface name="position">
-        <param name="initial_value">1.570796</param>
-      </state_interface>
-      </joint>
-      <joint name="${prefix}joint_a4">
-        <command_interface name="position"/>
-      <state_interface name="position">
-        <param name="initial_value">0.0</param>
-      </state_interface>
-      </joint>
-      <joint name="${prefix}joint_a5">
-        <command_interface name="position"/>
-      <state_interface name="position">
-        <param name="initial_value">0.0</param>
-      </state_interface>
-      </joint>
-      <joint name="${prefix}joint_a6">
-        <command_interface name="position"/>
-      <state_interface name="position">
-        <param name="initial_value">0.0</param>
-      </state_interface>
-      </joint>
-    </ros2_control>
   </xacro:macro>
 </robot>

File: kuka_resources/urdf/common_colours.xacro (robot description, xacro)
@@ -9,5 +9,5 @@
   <!-- default colors for robots -->
   <!-- RAL 2003: mechanical arm (pastel orange) -->
-  <xacro:property name="colour_kuka_orange"               value="${246/255} ${120/255} ${ 40/255} 1.0" />
+  <xacro:property name="colour_kuka_orange"               value="${246/255} ${120/255} ${ 40/255} 0.5" />
   <!-- RAL 9005: robot base (jet black) -->
   <xacro:property name="colour_kuka_black"                value="${ 14/255} ${ 14/255} ${ 16/255} 1.0" />
