Commit message: Fixed bug in kr150_r3100-2 urdf

File: kuka_quantec_support/urdf/kr150_r3100-2.urdf.xacro (robot description, xacro)
@@ -8,15 +8,40 @@
   <xacro:property name="client_port" value="${rsi_config_dict['client_port']}" /> -->
   <!-- Read additional arguments  -->
-  <xacro:arg name="use_fake_hardware" default="false" />
+  <!-- <xacro:arg name="use_fake_hardware" default="false" />
   <xacro:arg name="rsi_config_file" default="rsi_config.yaml" />
-  <xacro:arg name="namespace" default="" />
+  <xacro:arg name="namespace" default="" /> -->
   <!-- Turn the rsi config file argument into a property, for comparison -->
   <!-- <xacro:property name="default_rsi_config_file" value="rsi_config.yaml"/> -->
   <!-- <xacro:property name="current_rsi_config_file" value="$(arg rsi_config_file)"/> -->
   <!-- Read parameters from rsi_config  -->
-  <xacro:property name="rsi_config" value="$(arg rsi_config_file)" />
+  <!-- <xacro:property name="rsi_config" value="$(arg rsi_config_file)" />
   <xacro:property name="rsi_config_dict" value="${xacro.load_yaml(rsi_config)}"/>
   <xacro:property name="client_ip" value="${rsi_config_dict['client_ip']}"/>
-  <xacro:property name="client_port" value="${rsi_config_dict['client_port']}" />
+  <xacro:property name="client_port" value="${rsi_config_dict['client_port']}" /> -->
+<!-- Read additional arguments  -->
+<xacro:arg name="use_fake_hardware" default="false" />
+<xacro:arg name="rsi_config_file" default="rsi_config.yaml" />
+<xacro:arg name="namespace" default="" />
+<xacro:property name="use_fake_hardware_prop" value="$(arg use_fake_hardware)"/>
+<xacro:property name="false_prop" value="false"/>
+<xacro:unless value="${use_fake_hardware_prop == false_prop}">
+    <!-- Turn the rsi config file argument into a property, for comparison-->
+    <xacro:property name="default_rsi_config_file" value="rsi_config.yaml"/>
+    <xacro:property name="current_rsi_config_file" value="$(arg rsi_config_file)"/>
+    <!-- Read parameters from rsi_config  -->
+    <xacro:property name="rsi_config" value="$(arg rsi_config_file)" />
+    <xacro:if value="${current_rsi_config_file == default_rsi_config_file}">
+        <xacro:property name="rsi_config_dict" value="${xacro.load_yaml(rsi_config)}"/>
+    </xacro:if>
+    <xacro:unless value="${current_rsi_config_file == default_rsi_config_file}">
+        <xacro:property name="rsi_config_dict" value="${xacro.load_yaml(rsi_config)}"/>
+    </xacro:unless>
+    <xacro:property name="client_ip" value="${rsi_config_dict['client_ip']}"/>
+    <xacro:property name="client_port" value="${rsi_config_dict['client_port']}" />
+</xacro:unless>
+<xacro:if value="${use_fake_hardware_prop == false_prop}">
+    <xacro:property name="client_ip" value="0.0.0.0"/>
+    <xacro:property name="client_port" value="0" />
+</xacro:if>
   <xacro:kuka_kr150_r3100-2_robot prefix="$(arg namespace)"
                   client_ip="${client_ip}"
