Commit message: fix the UR flange orientation

File: kuka_quantec_support/urdf/kr150_r3100-2_macro.xacro (robot description, xacro)
@@ -263,5 +263,8 @@
     <link name="${prefix}flange" />
     <joint name="${prefix}joint_6-flange" type="fixed">
-      <origin xyz="0 0 0" rpy="0 0 0" />
+    <!-- ORIGINAL -->
+      <!-- <origin xyz="0 0 0" rpy="0 0 0" /> -->
+    <!-- After the Fine Tube Validation using LR and UR | 06102024 -->
+      <origin xyz="0 0 0" rpy="-0.0122173 0 0" />
       <parent link="${prefix}link_6" />
       <child link="${prefix}flange" />

Commit message: Revert "fix the UR flange orientation"
This reverts commit c9d7915459209b93113697e92bd68f473b2f94c8.

File: kuka_quantec_support/urdf/kr150_r3100-2_macro.xacro (robot description, xacro)
@@ -263,8 +263,5 @@
     <link name="${prefix}flange" />
     <joint name="${prefix}joint_6-flange" type="fixed">
-    <!-- ORIGINAL -->
-      <!-- <origin xyz="0 0 0" rpy="0 0 0" /> -->
-    <!-- After the Fine Tube Validation using LR and UR | 06102024 -->
-      <origin xyz="0 0 0" rpy="-0.0122173 0 0" />
+      <origin xyz="0 0 0" rpy="0 0 0" />
       <parent link="${prefix}link_6" />
       <child link="${prefix}flange" />
