Commit message: Put external axis last for proper RSI driver order

File: kuka_cybertech_support/urdf/kr_cybertech_ros2_control_macro.xacro (robot description, xacro)
@@ -32,12 +32,4 @@
         </xacro:if>
       </hardware>
-      <xacro:if value="${external_axis}">
-        <joint name="${prefix}linear_rail">
-          <command_interface name="position"/>
-          <state_interface name="position">
-            <param name="initial_value">0.0</param>
-          </state_interface>
-        </joint>
-      </xacro:if>
       <joint name="${prefix}joint_1">
         <command_interface name="position"/>
@@ -76,4 +68,12 @@
         </state_interface>
       </joint>
+      <xacro:if value="${external_axis}">
+        <joint name="${prefix}linear_rail">
+          <command_interface name="position"/>
+          <state_interface name="position">
+            <param name="initial_value">0.0</param>
+          </state_interface>
+        </joint>
+      </xacro:if>
       <xacro:if value="${use_gpio}">
         <xacro:include filename="$(find kuka_rsi_driver)/config/gpio_config.xacro"/>
