Commit message: Remove world link from cybertech macro, use parent argument instead

File: kuka_cybertech_support/urdf/kr16_r2010_2.urdf.xacro (robot description, xacro)
@@ -21,5 +21,6 @@
   <xacro:arg name="yaw" default="0"/>
   <xacro:kuka_cybertech_ros2_control name="$(arg prefix)kr16_r2010_2" driver_version="$(arg driver_version)" client_ip="$(arg client_ip)" client_port="$(arg client_port)" controller_ip="$(arg controller_ip)" prefix="$(arg prefix)" mode="$(arg mode)" use_gpio="$(arg use_gpio)" roundtrip_time="$(arg roundtrip_time)" verify_robot_model="$(arg verify_robot_model)"/>
-  <xacro:kuka_kr16_r2010_2_robot prefix="$(arg prefix)" package_name="kuka_cybertech_support">
+  <link name="world" />
+  <xacro:kuka_kr16_r2010_2_robot prefix="$(arg prefix)" package_name="kuka_cybertech_support" parent="world">
     <origin xyz="$(arg x) $(arg y) $(arg z)" rpy="$(arg roll) $(arg pitch) $(arg yaw)"/>
   </xacro:kuka_kr16_r2010_2_robot>

File: kuka_cybertech_support/urdf/kr16_r2010_2_macro.xacro (robot description, xacro)
@@ -1,7 +1,6 @@
 <?xml version="1.0"?>
 <robot xmlns:xacro="http://wiki.ros.org/xacro">
-  <xacro:macro name="kuka_kr16_r2010_2_robot" params="prefix package_name *origin">
+  <xacro:macro name="kuka_kr16_r2010_2_robot" params="prefix package_name *origin parent">
     <!-- links - main serial chain -->
-    <link name="world"/>
     <link name="${prefix}base_link">
       <collision>
@@ -102,6 +101,6 @@
       </visual>
     </link>
-    <joint name="${prefix}world-base_link" type="fixed">
-      <parent link="world"/>
+    <joint name="${prefix}parent-base_link" type="fixed">
+      <parent link="${parent}"/>
       <child link="${prefix}base_link"/>
       <xacro:insert_block name="origin"/>

Commit message: Fix pre-commit

File: kuka_cybertech_support/urdf/kr16_r2010_2.urdf.xacro (robot description, xacro)
@@ -21,5 +21,5 @@
   <xacro:arg name="yaw" default="0"/>
   <xacro:kuka_cybertech_ros2_control name="$(arg prefix)kr16_r2010_2" driver_version="$(arg driver_version)" client_ip="$(arg client_ip)" client_port="$(arg client_port)" controller_ip="$(arg controller_ip)" prefix="$(arg prefix)" mode="$(arg mode)" use_gpio="$(arg use_gpio)" roundtrip_time="$(arg roundtrip_time)" verify_robot_model="$(arg verify_robot_model)"/>
-  <link name="world" />
+  <link name="world"/>
   <xacro:kuka_kr16_r2010_2_robot prefix="$(arg prefix)" package_name="kuka_cybertech_support" parent="world">
     <origin xyz="$(arg x) $(arg y) $(arg z)" rpy="$(arg roll) $(arg pitch) $(arg yaw)"/>

File: kuka_cybertech_support/urdf/kr16_r2010_2_macro.xacro (robot description, xacro)
@@ -5,16 +5,16 @@
       <link name="${prefix}rail_base">
         <visual>
-          <origin rpy="0 0 0" xyz="-4.6875 0 0" />
-          <geometry>
-            <mesh filename="package://${package_name}/meshes/kr16_r2010_2/visual/rail_base.stl" scale="1 1 1" />
+          <origin rpy="0 0 0" xyz="-4.6875 0 0"/>
+          <geometry>
+            <mesh filename="package://${package_name}/meshes/kr16_r2010_2/visual/rail_base.stl" scale="1 1 1"/>
           </geometry>
           <material name="grey">
-            <color rgba="0.1 0.1 0.1 1.0" />
+            <color rgba="0.1 0.1 0.1 1.0"/>
           </material>
         </visual>
         <collision>
-          <origin rpy="0 0 0" xyz="-4.6875 0 0" />
-          <geometry>
-            <mesh filename="package://${package_name}/meshes/kr16_r2010_2/collision/rail_base.stl" scale="1 1 1" />
+          <origin rpy="0 0 0" xyz="-4.6875 0 0"/>
+          <geometry>
+            <mesh filename="package://${package_name}/meshes/kr16_r2010_2/collision/rail_base.stl" scale="1 1 1"/>
           </geometry>
         </collision>
@@ -23,17 +23,16 @@
         <visual>
           <!-- TODO eyeballed this origin, needs to be measured -->
-          <origin rpy="0 0 0" xyz="-0.4975 0 0" />
-          <geometry>
-            <mesh filename="package://${package_name}/meshes/kr16_r2010_2/visual/rail_carriage.stl" scale="1 1 1" />
+          <origin rpy="0 0 0" xyz="-0.4975 0 0"/>
+          <geometry>
+            <mesh filename="package://${package_name}/meshes/kr16_r2010_2/visual/rail_carriage.stl" scale="1 1 1"/>
           </geometry>
           <material name="light_grey">
-            <color rgba="0.6 0.6 0.6 1.0" />
+            <color rgba="0.6 0.6 0.6 1.0"/>
           </material>
         </visual>
         <collision>
-          <origin rpy="0 0 0" xyz="-0.4975 0 0" />
-          <geometry>
-            <mesh filename="package://${package_name}/meshes/kr16_r2010_2/collision/rail_carriage.stl"
-              scale="1 1 1" />
+          <origin rpy="0 0 0" xyz="-0.4975 0 0"/>
+          <geometry>
+            <mesh filename="package://${package_name}/meshes/kr16_r2010_2/collision/rail_carriage.stl" scale="1 1 1"/>
           </geometry>
         </collision>
@@ -141,19 +140,19 @@
     <xacro:if value="${external_axis}">
       <joint name="${prefix}parent-rail_base" type="fixed">
-        <parent link="${parent}" />
-        <child link="${prefix}rail_base" />
+        <parent link="${parent}"/>
+        <child link="${prefix}rail_base"/>
         <xacro:insert_block name="origin"/>
       </joint>
       <joint name="${prefix}linear_rail" type="prismatic">
-        <axis xyz="1 0 0" />
-        <parent link="${prefix}rail_base" />
-        <child link="${prefix}rail_carriage" />
-        <origin rpy="0 0 0" xyz="0 0 0" />
-        <limit acceleration="0.5" effort="100000.0" lower="-3.0" upper="3.0" velocity="0.175" />
+        <axis xyz="1 0 0"/>
+        <parent link="${prefix}rail_base"/>
+        <child link="${prefix}rail_carriage"/>
+        <origin rpy="0 0 0" xyz="0 0 0"/>
+        <limit acceleration="0.5" effort="100000.0" lower="-3.0" upper="3.0" velocity="0.175"/>
       </joint>
       <joint name="${prefix}base_link" type="fixed">
         <parent link="${prefix}rail_carriage"/>
         <child link="${prefix}base_link"/>
-        <origin xyz="0 0.159 0" rpy="-1.5708 -1.5708 0" />
+        <origin xyz="0 0.159 0" rpy="-1.5708 -1.5708 0"/>
       </joint>
     </xacro:if>

Commit message: Add new gpio_config_file instead to replace use_gpio

File: kuka_cybertech_support/urdf/kr16_r2010_2.urdf.xacro (robot description, xacro)
@@ -7,5 +7,5 @@
   <xacro:arg name="driver_version" default="eki_rsi"/>
   <xacro:arg name="mode" default="hardware"/>
-  <xacro:arg name="use_gpio" default="false"/>
+  <xacro:arg name="gpio_config_file" default=""/>
   <xacro:arg name="roundtrip_time" default="0"/>
   <xacro:arg name="client_ip" default="0.0.0.0"/>
@@ -21,5 +21,5 @@
   <xacro:arg name="yaw" default="0"/>
   <xacro:arg name="external_axis" default="false"/>
-  <xacro:kuka_cybertech_ros2_control name="$(arg prefix)kr16_r2010_2" driver_version="$(arg driver_version)" client_ip="$(arg client_ip)" client_port="$(arg client_port)" controller_ip="$(arg controller_ip)" prefix="$(arg prefix)" mode="$(arg mode)" use_gpio="$(arg use_gpio)" roundtrip_time="$(arg roundtrip_time)" verify_robot_model="$(arg verify_robot_model)"/>
+  <xacro:kuka_cybertech_ros2_control name="$(arg prefix)kr16_r2010_2" driver_version="$(arg driver_version)" client_ip="$(arg client_ip)" client_port="$(arg client_port)" controller_ip="$(arg controller_ip)" prefix="$(arg prefix)" mode="$(arg mode)" gpio_config_file="$(arg gpio_config_file)" roundtrip_time="$(arg roundtrip_time)" verify_robot_model="$(arg verify_robot_model)"/>
   <link name="world"/>
   <xacro:kuka_kr16_r2010_2_robot prefix="$(arg prefix)" package_name="kuka_cybertech_support" parent="world" external_axis="$(arg external_axis)">

File: kuka_cybertech_support/urdf/kr_cybertech_ros2_control_macro.xacro (robot description, xacro)
@@ -1,5 +1,5 @@
 <?xml version="1.0" encoding="UTF-8"?>
 <robot xmlns:xacro="http://www.ros.org/wiki/xacro">
-  <xacro:macro name="kuka_cybertech_ros2_control" params="name driver_version client_ip client_port controller_ip prefix mode use_gpio roundtrip_time verify_robot_model external_axis:=false">
+  <xacro:macro name="kuka_cybertech_ros2_control" params="name driver_version client_ip client_port controller_ip prefix mode gpio_config_file:='' roundtrip_time verify_robot_model external_axis:=false">
     <!-- gazebo -->
     <xacro:if value="${mode == 'gazebo'}">
@@ -99,9 +99,9 @@
         </joint>
       </xacro:if>
-      <xacro:if value="${use_gpio}">
-        <xacro:include filename="$(find kuka_rsi_driver)/config/gpio_config.xacro"/>
+      <xacro:if value="${gpio_config_file != ''}">
+        <xacro:include filename="${gpio_config_file}"/>
         <xacro:gpio_config prefix="${prefix}"/>
       </xacro:if>
-      <xacro:unless value="${use_gpio}">
+      <xacro:unless value="${gpio_config_file != ''}">
         <gpio name="gpio"/>
       </xacro:unless>
