Commit message: Add optional external linear axis to cybertech macros

File: kuka_cybertech_support/urdf/kr16_r2010_2_macro.xacro (robot description, xacro)
@@ -1,5 +1,43 @@
 <?xml version="1.0"?>
 <robot xmlns:xacro="http://wiki.ros.org/xacro">
-  <xacro:macro name="kuka_kr16_r2010_2_robot" params="prefix package_name *origin parent">
+  <xacro:macro name="kuka_kr16_r2010_2_robot" params="prefix package_name *origin parent external_axis:=false">
+    <xacro:if value="${external_axis}">
+      <link name="${prefix}rail_base">
+        <visual>
+          <origin rpy="0 0 0" xyz="-4.6875 0 0" />
+          <geometry>
+            <mesh filename="package://${package_name}/meshes/kr16_r2010_2/visual/rail_base.stl" scale="1 1 1" />
+          </geometry>
+          <material name="grey">
+            <color rgba="0.1 0.1 0.1 1.0" />
+          </material>
+        </visual>
+        <collision>
+          <origin rpy="0 0 0" xyz="-4.6875 0 0" />
+          <geometry>
+            <mesh filename="package://${package_name}/meshes/kr16_r2010_2/collision/rail_base.stl" scale="1 1 1" />
+          </geometry>
+        </collision>
+      </link>
+      <link name="${prefix}rail_carriage">
+        <visual>
+          <!-- TODO eyeballed this origin, needs to be measured -->
+          <origin rpy="0 0 0" xyz="-0.4975 0 0" />
+          <geometry>
+            <mesh filename="package://${package_name}/meshes/kr16_r2010_2/visual/rail_carriage.stl" scale="1 1 1" />
+          </geometry>
+          <material name="light_grey">
+            <color rgba="0.6 0.6 0.6 1.0" />
+          </material>
+        </visual>
+        <collision>
+          <origin rpy="0 0 0" xyz="-0.4975 0 0" />
+          <geometry>
+            <mesh filename="package://${package_name}/meshes/kr16_r2010_2/collision/rail_carriage.stl"
+              scale="1 1 1" />
+          </geometry>
+        </collision>
+      </link>
+    </xacro:if>
     <!-- links - main serial chain -->
     <link name="${prefix}base_link">
@@ -101,9 +139,30 @@
       </visual>
     </link>
-    <joint name="${prefix}parent-base_link" type="fixed">
-      <parent link="${parent}"/>
-      <child link="${prefix}base_link"/>
-      <xacro:insert_block name="origin"/>
-    </joint>
+    <xacro:if value="${external_axis}">
+      <joint name="${prefix}parent-rail_base" type="fixed">
+        <parent link="${parent}" />
+        <child link="${prefix}rail_base" />
+        <xacro:insert_block name="origin"/>
+      </joint>
+      <joint name="${prefix}linear_rail" type="prismatic">
+        <axis xyz="1 0 0" />
+        <parent link="${prefix}rail_base" />
+        <child link="${prefix}rail_carriage" />
+        <origin rpy="0 0 0" xyz="0 0 0" />
+        <limit acceleration="10.0" effort="1000.0" lower="-3.66" upper="3.66" velocity="0.175" />
+      </joint>
+      <joint name="${prefix}base_link" type="fixed">
+        <parent link="${prefix}rail_carriage"/>
+        <child link="${prefix}base_link"/>
+        <origin xyz="0 0.159 0" rpy="-1.5708 0 0" />
+      </joint>
+    </xacro:if>
+    <xacro:unless value="${external_axis}">
+      <joint name="${prefix}parent-base_link" type="fixed">
+        <parent link="${parent}"/>
+        <child link="${prefix}base_link"/>
+        <xacro:insert_block name="origin"/>
+      </joint>
+    </xacro:unless>
     <joint name="${prefix}joint_1" type="revolute">
       <axis xyz="0.0 0.0 1.0"/>

File: kuka_cybertech_support/urdf/kr_cybertech_ros2_control_macro.xacro (robot description, xacro)
@@ -1,5 +1,5 @@
 <?xml version="1.0" encoding="UTF-8"?>
 <robot xmlns:xacro="http://www.ros.org/wiki/xacro">
-  <xacro:macro name="kuka_cybertech_ros2_control" params="name driver_version client_ip client_port controller_ip prefix mode use_gpio roundtrip_time verify_robot_model">
+  <xacro:macro name="kuka_cybertech_ros2_control" params="name driver_version client_ip client_port controller_ip prefix mode use_gpio roundtrip_time verify_robot_model external_axis:=false">
     <!-- gazebo -->
     <xacro:if value="${mode == 'gazebo'}">
@@ -32,4 +32,12 @@
         </xacro:if>
       </hardware>
+      <xacro:if value="${external_axis}">
+        <joint name="${prefix}linear_rail">
+          <command_interface name="position"/>
+          <state_interface name="position">
+            <param name="initial_value">0.0</param>
+          </state_interface>
+        </joint>
+      </xacro:if>
       <joint name="${prefix}joint_1">
         <command_interface name="position"/>

Commit message: change orientation of arm

File: kuka_cybertech_support/urdf/kr16_r2010_2_macro.xacro (robot description, xacro)
@@ -150,10 +150,10 @@
         <child link="${prefix}rail_carriage" />
         <origin rpy="0 0 0" xyz="0 0 0" />
-        <limit acceleration="10.0" effort="1000.0" lower="-3.66" upper="3.66" velocity="0.175" />
+        <limit acceleration="1.0" effort="100000.0" lower="-2.0" upper="2.0" velocity="0.175" />
       </joint>
       <joint name="${prefix}base_link" type="fixed">
         <parent link="${prefix}rail_carriage"/>
         <child link="${prefix}base_link"/>
-        <origin xyz="0 0.159 0" rpy="-1.5708 0 0" />
+        <origin xyz="0 0.159 0" rpy="-1.5708 -1.5708 0" />
       </joint>
     </xacro:if>

Commit message: dress pack joint limit

File: kuka_cybertech_support/urdf/kr16_r2010_2_macro.xacro (robot description, xacro)
@@ -150,5 +150,5 @@
         <child link="${prefix}rail_carriage" />
         <origin rpy="0 0 0" xyz="0 0 0" />
-        <limit acceleration="1.0" effort="100000.0" lower="-2.0" upper="2.0" velocity="0.175" />
+        <limit acceleration="0.5" effort="100000.0" lower="-3.0" upper="3.0" velocity="0.175" />
       </joint>
       <joint name="${prefix}base_link" type="fixed">
@@ -175,5 +175,5 @@
       <axis xyz="0.0 0.0 1.0"/>
       <child link="${prefix}link_2"/>
-      <limit effort="1633.6259859" lower="-3.2288591161895095E0" upper="1.1344640137963142E0" velocity="${radians(175)}"/>
+      <limit effort="1633.6259859" lower="-3.01" upper="1.1344640137963142E0" velocity="${radians(175)}"/>
       <origin rpy="${pi/2.0} 0.0 -0.0" xyz="0.16 0.0 -0.52"/>
       <parent link="${prefix}link_1"/>

Commit message: remove TODO, fix arm joint limit

File: kuka_cybertech_support/urdf/kr16_r2010_2_macro.xacro (robot description, xacro)
@@ -22,5 +22,4 @@
       <link name="${prefix}rail_carriage">
         <visual>
-          <!-- TODO eyeballed this origin, needs to be measured -->
           <origin rpy="0 0 0" xyz="-0.4975 0 0"/>
           <geometry>
@@ -174,5 +173,5 @@
       <axis xyz="0.0 0.0 1.0"/>
       <child link="${prefix}link_2"/>
-      <limit effort="1633.6259859" lower="-3.01" upper="1.1344640137963142E0" velocity="${radians(175)}"/>
+      <limit effort="1633.6259859" lower="-3.2288591161895095E0" upper="1.1344640137963142E0" velocity="${radians(175)}"/>
       <origin rpy="${pi/2.0} 0.0 -0.0" xyz="0.16 0.0 -0.52"/>
       <parent link="${prefix}link_1"/>

Commit message: wip gpio

File: kuka_cybertech_support/urdf/kr16_r2010_2_macro.xacro (robot description, xacro)
@@ -148,5 +148,5 @@
         <child link="${prefix}rail_carriage"/>
         <origin rpy="0 0 0" xyz="0 0 0"/>
-        <limit acceleration="0.5" effort="100000.0" lower="-3.0" upper="3.0" velocity="0.175"/>
+        <limit acceleration="0.5" effort="100000.0" lower="-3.6" upper="3.8" velocity="0.175"/>
       </joint>
       <joint name="${prefix}base_link" type="fixed">

File: kuka_cybertech_support/urdf/kr_cybertech_ros2_control_macro.xacro (robot description, xacro)
@@ -101,5 +101,5 @@
       <xacro:if value="${use_gpio}">
         <xacro:include filename="$(find kuka_rsi_driver)/config/gpio_config.xacro"/>
-        <xacro:gpio_config/>
+        <xacro:gpio_config prefix="${prefix}"/>
       </xacro:if>
       <xacro:unless value="${use_gpio}">

Commit message: increase rail hardware limits

File: kuka_cybertech_support/urdf/kr16_r2010_2_macro.xacro (robot description, xacro)
@@ -148,5 +148,5 @@
         <child link="${prefix}rail_carriage"/>
         <origin rpy="0 0 0" xyz="0 0 0"/>
-        <limit acceleration="0.5" effort="100000.0" lower="-3.0" upper="3.0" velocity="0.175"/>
+        <limit acceleration="0.5" effort="100000.0" lower="-4.5" upper="4.5" velocity="0.175"/>
       </joint>
       <joint name="${prefix}base_link" type="fixed">

Commit message: Use convex hulls for collision meshes

File: kuka_cybertech_support/urdf/kr16_r2010_2_macro.xacro (robot description, xacro)
@@ -16,5 +16,5 @@
           <origin rpy="0 0 0" xyz="-4.6875 0 0"/>
           <geometry>
-            <mesh filename="package://${package_name}/meshes/kr16_r2010_2/collision/rail_base.stl" scale="1 1 1"/>
+            <mesh filename="package://${package_name}/meshes/kr16_r2010_2/collision/rail_base_convex.stl" scale="1 1 1"/>
           </geometry>
         </collision>
@@ -33,5 +33,5 @@
           <origin rpy="0 0 0" xyz="-0.4975 0 0"/>
           <geometry>
-            <mesh filename="package://${package_name}/meshes/kr16_r2010_2/collision/rail_carriage.stl" scale="1 1 1"/>
+            <mesh filename="package://${package_name}/meshes/kr16_r2010_2/collision/rail_carriage_convex.stl" scale="1 1 1"/>
           </geometry>
         </collision>
@@ -42,5 +42,5 @@
       <collision>
         <geometry>
-          <mesh filename="package://${package_name}/meshes/kr16_r2010_2/collision/base_link.stl"/>
+          <mesh filename="package://${package_name}/meshes/kr16_r2010_2/collision/base_link_convex.stl"/>
         </geometry>
         <origin rpy="-0.0 0.0 -0.0" xyz="0.0 0.0 0.0"/>
@@ -56,5 +56,5 @@
       <collision>
         <geometry>
-          <mesh filename="package://${package_name}/meshes/kr16_r2010_2/collision/link_1.stl"/>
+          <mesh filename="package://${package_name}/meshes/kr16_r2010_2/collision/link_1_convex.stl"/>
         </geometry>
         <origin rpy="-0.0 0.0 -0.0" xyz="0.0 0.0 0.0"/>
@@ -70,5 +70,5 @@
       <collision>
         <geometry>
-          <mesh filename="package://${package_name}/meshes/kr16_r2010_2/collision/link_2.stl"/>
+          <mesh filename="package://${package_name}/meshes/kr16_r2010_2/collision/link_2_convex.stl"/>
         </geometry>
         <origin rpy="-0.0 0.0 -0.0" xyz="0.0 0.0 0.0"/>
@@ -84,5 +84,5 @@
       <collision>
         <geometry>
-          <mesh filename="package://${package_name}/meshes/kr16_r2010_2/collision/link_3.stl"/>
+          <mesh filename="package://${package_name}/meshes/kr16_r2010_2/collision/link_3_convex.stl"/>
         </geometry>
         <origin rpy="-0.0 0.0 -0.0" xyz="0.0 0.0 0.0"/>
@@ -98,5 +98,5 @@
       <collision>
         <geometry>
-          <mesh filename="package://${package_name}/meshes/kr16_r2010_2/collision/link_4.stl"/>
+          <mesh filename="package://${package_name}/meshes/kr16_r2010_2/collision/link_4_convex.stl"/>
         </geometry>
         <origin rpy="-0.0 0.0 -0.0" xyz="0.0 0.0 0.0"/>
@@ -112,5 +112,5 @@
       <collision>
         <geometry>
-          <mesh filename="package://${package_name}/meshes/kr16_r2010_2/collision/link_5.stl"/>
+          <mesh filename="package://${package_name}/meshes/kr16_r2010_2/collision/link_5_convex.stl"/>
         </geometry>
         <origin rpy="-0.0 0.0 -0.0" xyz="0.0 0.0 0.0"/>
@@ -126,5 +126,5 @@
       <collision>
         <geometry>
-          <mesh filename="package://${package_name}/meshes/kr16_r2010_2/collision/link_6.stl"/>
+          <mesh filename="package://${package_name}/meshes/kr16_r2010_2/collision/link_6_convex.stl"/>
         </geometry>
         <origin rpy="-0.0 0.0 -0.0" xyz="0.0 0.0 0.0"/>

Commit message: split link 4 into 2 pieces

File: kuka_cybertech_support/urdf/kr16_r2010_2_macro.xacro (robot description, xacro)
@@ -98,14 +98,22 @@
       <collision>
         <geometry>
+          <mesh filename="package://${package_name}/meshes/kr16_r2010_2/collision/link_4_part_1.stl"/>
+        </geometry>
+        <origin rpy="-0.0 0.0 -0.0" xyz="0.0 0.0 0.0"/>
+      </collision>
+      <visual>
+        <geometry>
+          <mesh filename="package://${package_name}/meshes/kr16_r2010_2/visual/link_4.stl"/>
+        </geometry>
+        <origin rpy="-0.0 0.0 -0.0" xyz="0.0 0.0 0.0"/>
+      </visual>
+    </link>
+    <link name="${prefix}link_4_part_2">
+      <collision>
+        <geometry>
           <mesh filename="package://${package_name}/meshes/kr16_r2010_2/collision/link_4.stl"/>
         </geometry>
         <origin rpy="-0.0 0.0 -0.0" xyz="0.0 0.0 0.0"/>
       </collision>
-      <visual>
-        <geometry>
-          <mesh filename="package://${package_name}/meshes/kr16_r2010_2/visual/link_4.stl"/>
-        </geometry>
-        <origin rpy="-0.0 0.0 -0.0" xyz="0.0 0.0 0.0"/>
-      </visual>
     </link>
     <link name="${prefix}link_5">
@@ -191,4 +199,9 @@
       <parent link="${prefix}link_3"/>
     </joint>
+    <joint name="${prefix}joint_4_middle" type="fixed">
+      <child link="${prefix}link_4_part_2"/>
+      <origin rpy="0.0 0.0 -0.0" xyz="0.0 0.0 0.0"/>
+      <parent link="${prefix}link_4"/>
+    </joint>
     <joint name="${prefix}joint_5" type="revolute">
       <axis xyz="0.0 0.0 1.0"/>

Commit message: Add convex meshes

File: kuka_cybertech_support/urdf/kr16_r2010_2_macro.xacro (robot description, xacro)
@@ -16,5 +16,5 @@
           <origin rpy="0 0 0" xyz="-4.6875 0 0"/>
           <geometry>
-            <mesh filename="package://${package_name}/meshes/kr16_r2010_2/collision/rail_base.stl" scale="1 1 1"/>
+            <mesh filename="package://${package_name}/meshes/kr16_r2010_2/collision/rail_base_convex.stl" scale="1 1 1"/>
           </geometry>
         </collision>
@@ -33,5 +33,5 @@
           <origin rpy="0 0 0" xyz="-0.4975 0 0"/>
           <geometry>
-            <mesh filename="package://${package_name}/meshes/kr16_r2010_2/collision/rail_carriage.stl" scale="1 1 1"/>
+            <mesh filename="package://${package_name}/meshes/kr16_r2010_2/collision/rail_carriage_convex.stl" scale="1 1 1"/>
           </geometry>
         </collision>
@@ -42,5 +42,5 @@
       <collision>
         <geometry>
-          <mesh filename="package://${package_name}/meshes/kr16_r2010_2/collision/base_link.stl"/>
+          <mesh filename="package://${package_name}/meshes/kr16_r2010_2/collision/base_link_convex.stl"/>
         </geometry>
         <origin rpy="-0.0 0.0 -0.0" xyz="0.0 0.0 0.0"/>
@@ -56,5 +56,5 @@
       <collision>
         <geometry>
-          <mesh filename="package://${package_name}/meshes/kr16_r2010_2/collision/link_1.stl"/>
+          <mesh filename="package://${package_name}/meshes/kr16_r2010_2/collision/link_1_convex.stl"/>
         </geometry>
         <origin rpy="-0.0 0.0 -0.0" xyz="0.0 0.0 0.0"/>
@@ -70,5 +70,5 @@
       <collision>
         <geometry>
-          <mesh filename="package://${package_name}/meshes/kr16_r2010_2/collision/link_2.stl"/>
+          <mesh filename="package://${package_name}/meshes/kr16_r2010_2/collision/link_2_convex.stl"/>
         </geometry>
         <origin rpy="-0.0 0.0 -0.0" xyz="0.0 0.0 0.0"/>
@@ -84,5 +84,5 @@
       <collision>
         <geometry>
-          <mesh filename="package://${package_name}/meshes/kr16_r2010_2/collision/link_3.stl"/>
+          <mesh filename="package://${package_name}/meshes/kr16_r2010_2/collision/link_3_convex.stl"/>
         </geometry>
         <origin rpy="-0.0 0.0 -0.0" xyz="0.0 0.0 0.0"/>
@@ -98,5 +98,5 @@
       <collision>
         <geometry>
-          <mesh filename="package://${package_name}/meshes/kr16_r2010_2/collision/link_4_part_1.stl"/>
+          <mesh filename="package://${package_name}/meshes/kr16_r2010_2/collision/link_4_part_1_convex.stl"/>
         </geometry>
         <origin rpy="-0.0 0.0 -0.0" xyz="0.0 0.0 0.0"/>
@@ -112,5 +112,5 @@
       <collision>
         <geometry>
-          <mesh filename="package://${package_name}/meshes/kr16_r2010_2/collision/link_4.stl"/>
+          <mesh filename="package://${package_name}/meshes/kr16_r2010_2/collision/link_4_convex.stl"/>
         </geometry>
         <origin rpy="-0.0 0.0 -0.0" xyz="0.0 0.0 0.0"/>
@@ -120,5 +120,5 @@
       <collision>
         <geometry>
-          <mesh filename="package://${package_name}/meshes/kr16_r2010_2/collision/link_5.stl"/>
+          <mesh filename="package://${package_name}/meshes/kr16_r2010_2/collision/link_5_convex.stl"/>
         </geometry>
         <origin rpy="-0.0 0.0 -0.0" xyz="0.0 0.0 0.0"/>
@@ -134,5 +134,5 @@
       <collision>
         <geometry>
-          <mesh filename="package://${package_name}/meshes/kr16_r2010_2/collision/link_6.stl"/>
+          <mesh filename="package://${package_name}/meshes/kr16_r2010_2/collision/link_6_convex.stl"/>
         </geometry>
         <origin rpy="-0.0 0.0 -0.0" xyz="0.0 0.0 0.0"/>

Commit message: update colors

File: kuka_cybertech_support/urdf/kr16_r2010_2_macro.xacro (robot description, xacro)
@@ -26,6 +26,6 @@
             <mesh filename="package://${package_name}/meshes/kr16_r2010_2/visual/rail_carriage.stl" scale="1 1 1"/>
           </geometry>
-          <material name="light_grey">
-            <color rgba="0.6 0.6 0.6 1.0"/>
+          <material name="black">
+            <color rgba="0.05 0.05 0.05 1.0"/>
           </material>
         </visual>
@@ -51,4 +51,7 @@
         </geometry>
         <origin rpy="-0.0 0.0 -0.0" xyz="0.0 0.0 0.0"/>
+        <material name="orange">
+          <color rgba="0.7 0.18 0.0 1.0"/>
+        </material>
       </visual>
     </link>
@@ -65,4 +68,7 @@
         </geometry>
         <origin rpy="-0.0 0.0 -0.0" xyz="0.0 0.0 0.0"/>
+        <material name="orange">
+          <color rgba="0.7 0.18 0.0 1.0"/>
+        </material>
       </visual>
     </link>
@@ -79,4 +85,7 @@
         </geometry>
         <origin rpy="-0.0 0.0 -0.0" xyz="0.0 0.0 0.0"/>
+        <material name="orange">
+          <color rgba="0.7 0.18 0.0 1.0"/>
+        </material>
       </visual>
     </link>
@@ -93,4 +102,7 @@
         </geometry>
         <origin rpy="-0.0 0.0 -0.0" xyz="0.0 0.0 0.0"/>
+        <material name="orange">
+          <color rgba="0.7 0.18 0.0 1.0"/>
+        </material>
       </visual>
     </link>
@@ -107,4 +119,7 @@
         </geometry>
         <origin rpy="-0.0 0.0 -0.0" xyz="0.0 0.0 0.0"/>
+        <material name="orange">
+          <color rgba="0.7 0.18 0.0 1.0"/>
+        </material>
       </visual>
     </link>
@@ -129,4 +144,7 @@
         </geometry>
         <origin rpy="-0.0 0.0 -0.0" xyz="0.0 0.0 0.0"/>
+        <material name="orange">
+          <color rgba="0.7 0.18 0.0 1.0"/>
+        </material>
       </visual>
     </link>
@@ -143,4 +161,7 @@
         </geometry>
         <origin rpy="-0.0 0.0 -0.0" xyz="0.0 0.0 0.0"/>
+        <material name="orange">
+          <color rgba="0.7 0.18 0.0 1.0"/>
+        </material>
       </visual>
     </link>

Commit message: mirror axes

File: kuka_cybertech_support/urdf/kr16_r2010_2_macro.xacro (robot description, xacro)
@@ -1,5 +1,5 @@
 <?xml version="1.0"?>
 <robot xmlns:xacro="http://wiki.ros.org/xacro">
-  <xacro:macro name="kuka_kr16_r2010_2_robot" params="prefix package_name *origin parent external_axis:=false">
+  <xacro:macro name="kuka_kr16_r2010_2_robot" params="prefix package_name *origin parent external_axis:=false mirrored:=false">
     <xacro:if value="${external_axis}">
       <link name="${prefix}rail_base">
@@ -24,5 +24,10 @@
           <origin rpy="0 0 0" xyz="-0.4975 0 0"/>
           <geometry>
+            <xacro:unless value="${mirrored}">
             <mesh filename="package://${package_name}/meshes/kr16_r2010_2/visual/rail_carriage.stl" scale="1 1 1"/>
+            </xacro:unless>
+            <xacro:if value="${mirrored}">
+            <mesh filename="package://${package_name}/meshes/kr16_r2010_2/visual/rail_carriage_mirrored.stl" scale="1 1 1"/>
+            </xacro:if>
           </geometry>
           <material name="black">
@@ -33,5 +38,10 @@
           <origin rpy="0 0 0" xyz="-0.4975 0 0"/>
           <geometry>
+            <xacro:unless value="${mirrored}">
             <mesh filename="package://${package_name}/meshes/kr16_r2010_2/collision/rail_carriage_convex.stl" scale="1 1 1"/>
+            </xacro:unless>
+            <xacro:if value="${mirrored}">
+            <mesh filename="package://${package_name}/meshes/kr16_r2010_2/collision/rail_carriage_convex_mirrored.stl" scale="1 1 1"/>
+            </xacro:if>
           </geometry>
         </collision>

Commit message: pad rails a 10% (5% on each side)

File: kuka_cybertech_support/urdf/kr16_r2010_2_macro.xacro (robot description, xacro)
@@ -16,5 +16,5 @@
           <origin rpy="0 0 0" xyz="-4.6875 0 0"/>
           <geometry>
-            <mesh filename="package://${package_name}/meshes/kr16_r2010_2/collision/rail_base_convex.stl" scale="1 1 1"/>
+            <mesh filename="package://${package_name}/meshes/kr16_r2010_2/collision/rail_base_convex.stl" scale="1.1 1.1 1.1"/>
           </geometry>
         </collision>
@@ -39,8 +39,8 @@
           <geometry>
             <xacro:unless value="${mirrored}">
-            <mesh filename="package://${package_name}/meshes/kr16_r2010_2/collision/rail_carriage_convex.stl" scale="1 1 1"/>
+            <mesh filename="package://${package_name}/meshes/kr16_r2010_2/collision/rail_carriage_convex.stl" scale="1.1 1.1 1.1"/>
             </xacro:unless>
             <xacro:if value="${mirrored}">
-            <mesh filename="package://${package_name}/meshes/kr16_r2010_2/collision/rail_carriage_convex_mirrored.stl" scale="1 1 1"/>
+            <mesh filename="package://${package_name}/meshes/kr16_r2010_2/collision/rail_carriage_convex_mirrored.stl" scale="1.1 1.1 1.1"/>
             </xacro:if>
           </geometry>

Commit message: only scale y axis

File: kuka_cybertech_support/urdf/kr16_r2010_2_macro.xacro (robot description, xacro)
@@ -16,5 +16,5 @@
           <origin rpy="0 0 0" xyz="-4.6875 0 0"/>
           <geometry>
-            <mesh filename="package://${package_name}/meshes/kr16_r2010_2/collision/rail_base_convex.stl" scale="1.1 1.1 1.1"/>
+            <mesh filename="package://${package_name}/meshes/kr16_r2010_2/collision/rail_base_convex.stl" scale="1.0 1.1 1.0"/>
           </geometry>
         </collision>
@@ -39,8 +39,8 @@
           <geometry>
             <xacro:unless value="${mirrored}">
-            <mesh filename="package://${package_name}/meshes/kr16_r2010_2/collision/rail_carriage_convex.stl" scale="1.1 1.1 1.1"/>
+            <mesh filename="package://${package_name}/meshes/kr16_r2010_2/collision/rail_carriage_convex.stl" scale="1.0 1.1 1.0"/>
             </xacro:unless>
             <xacro:if value="${mirrored}">
-            <mesh filename="package://${package_name}/meshes/kr16_r2010_2/collision/rail_carriage_convex_mirrored.stl" scale="1.1 1.1 1.1"/>
+            <mesh filename="package://${package_name}/meshes/kr16_r2010_2/collision/rail_carriage_convex_mirrored.stl" scale="1.0 1.1 1.0"/>
             </xacro:if>
           </geometry>
