Commit message: Refactor KR16 rail kinematic chain with intermediate frames for site bringup: - Removes use of origin as the left rail carriage's zero point - Add explicit left/right rail_zero links relative to a more measurable origin point - Add explicit left/right rail_to_carriage_mount links relative to a more measurable origin point - Move hardcoded mesh offsets (e.g. -4.6875, -0.4975) from  visual/collision origins into joint transforms to promote tf2 debugging

File: kuka_cybertech_support/urdf/kr16_r2010_2_macro.xacro (robot description, xacro)
@@ -1,9 +1,27 @@
 <?xml version="1.0"?>
 <robot xmlns:xacro="http://wiki.ros.org/xacro">
-  <xacro:macro name="kuka_kr16_r2010_2_robot" params="prefix package_name *origin parent external_axis:=false mirrored:=false">
+  <xacro:macro name="kuka_kr16_r2010_2_robot" params="prefix package_name *origin parent external_axis:=false is_left:=false">
+    <!-- links - main serial chain -->
+    <link name="${prefix}base_link">
+      <collision>
+        <geometry>
+          <mesh filename="package://${package_name}/meshes/kr16_r2010_2/collision/base_link_convex.stl"/>
+        </geometry>
+        <origin rpy="-0.0 0.0 -0.0" xyz="0.0 0.0 0.0"/>
+      </collision>
+      <visual>
+        <geometry>
+          <mesh filename="package://${package_name}/meshes/kr16_r2010_2/visual/base_link.stl"/>
+        </geometry>
+        <origin rpy="-0.0 0.0 -0.0" xyz="0.0 0.0 0.0"/>
+        <material name="orange">
+          <color rgba="0.7 0.18 0.0 1.0"/>
+        </material>
+      </visual>
+    </link>
     <xacro:if value="${external_axis}">
+      <!-- Rail mesh origin is the center of left-most mounting bracket of the rail -->
       <link name="${prefix}rail_base">
         <visual>
-          <origin rpy="0 0 0" xyz="-4.6875 0 0"/>
           <geometry>
             <mesh filename="package://${package_name}/meshes/kr16_r2010_2/visual/rail_base.stl" scale="1 1 1"/>
@@ -14,5 +32,4 @@
         </visual>
         <collision>
-          <origin rpy="0 0 0" xyz="-4.6875 0 0"/>
           <geometry>
             <mesh filename="package://${package_name}/meshes/kr16_r2010_2/collision/rail_base_convex.stl" scale="1.0 1.1 1.0"/>
@@ -20,12 +37,37 @@
         </collision>
       </link>
-      <link name="${prefix}rail_carriage">
+      <joint name="${prefix}parent-rail_base" type="fixed">
+        <parent link="${parent}"/>
+        <child link="${prefix}rail_base"/>
+        <xacro:if value="${is_left}">
+          <origin xyz="0.315 0 0" rpy="3.141592 0 0"/>
+        </xacro:if>
+        <xacro:unless value="${is_left}">
+          <origin xyz="${(-4.288 - 0.850 - 4.870 + 0.315)} 0 0" rpy="3.141592 0 0"/>
+        </xacro:unless>
+      </joint>
+      <!-- The hand measured zero position of the "Kuka mounting pin" relative to the left-most point of the rail -->
+      <link name="${prefix}rail_zero"/>
+      <joint name="${prefix}rail_base-rail_zero" type="fixed">
+        <parent link="${parent}"/>
+        <child link="${prefix}rail_zero"/>
+        <xacro:insert_block name="origin"/>
+      </joint>
+      <!-- Inline with Kuka zero position -->
+      <link name="${prefix}rail_to_carriage_mount"/>
+      <joint name="${prefix}linear_rail" type="prismatic">
+        <axis xyz="1 0 0"/>
+        <parent link="${prefix}rail_zero"/>
+        <child link="${prefix}rail_to_carriage_mount"/>
+        <origin xyz="0 0 0" rpy="3.141592 0 0" />
+        <limit acceleration="0.5" effort="100000.0" lower="-4.5" upper="4.5" velocity="0.175"/>
+      </joint>
+      <link name="${prefix}rail_carriage_mesh">
         <visual>
-          <origin rpy="0 0 0" xyz="-0.4975 0 0"/>
-          <geometry>
-            <xacro:unless value="${mirrored}">
+          <geometry>
+            <xacro:unless value="${is_left}">
             <mesh filename="package://${package_name}/meshes/kr16_r2010_2/visual/rail_carriage.stl" scale="1 1 1"/>
             </xacro:unless>
-            <xacro:if value="${mirrored}">
+            <xacro:if value="${is_left}">
             <mesh filename="package://${package_name}/meshes/kr16_r2010_2/visual/rail_carriage_mirrored.stl" scale="1 1 1"/>
             </xacro:if>
@@ -36,10 +78,9 @@
         </visual>
         <collision>
-          <origin rpy="0 0 0" xyz="-0.4975 0 0"/>
-          <geometry>
-            <xacro:unless value="${mirrored}">
+          <geometry>
+            <xacro:unless value="${is_left}">
             <mesh filename="package://${package_name}/meshes/kr16_r2010_2/collision/rail_carriage_convex.stl" scale="1.0 1.1 1.0"/>
             </xacro:unless>
-            <xacro:if value="${mirrored}">
+            <xacro:if value="${is_left}">
             <mesh filename="package://${package_name}/meshes/kr16_r2010_2/collision/rail_carriage_convex_mirrored.stl" scale="1.0 1.1 1.0"/>
             </xacro:if>
@@ -47,150 +88,24 @@
         </collision>
       </link>
-    </xacro:if>
-    <!-- links - main serial chain -->
-    <link name="${prefix}base_link">
-      <collision>
-        <geometry>
-          <mesh filename="package://${package_name}/meshes/kr16_r2010_2/collision/base_link_convex.stl"/>
-        </geometry>
-        <origin rpy="-0.0 0.0 -0.0" xyz="0.0 0.0 0.0"/>
-      </collision>
-      <visual>
-        <geometry>
-          <mesh filename="package://${package_name}/meshes/kr16_r2010_2/visual/base_link.stl"/>
-        </geometry>
-        <origin rpy="-0.0 0.0 -0.0" xyz="0.0 0.0 0.0"/>
-        <material name="orange">
-          <color rgba="0.7 0.18 0.0 1.0"/>
-        </material>
-      </visual>
-    </link>
-    <link name="${prefix}link_1">
-      <collision>
-        <geometry>
-          <mesh filename="package://${package_name}/meshes/kr16_r2010_2/collision/link_1_convex.stl"/>
-        </geometry>
-        <origin rpy="-0.0 0.0 -0.0" xyz="0.0 0.0 0.0"/>
-      </collision>
-      <visual>
-        <geometry>
-          <mesh filename="package://${package_name}/meshes/kr16_r2010_2/visual/link_1.stl"/>
-        </geometry>
-        <origin rpy="-0.0 0.0 -0.0" xyz="0.0 0.0 0.0"/>
-        <material name="orange">
-          <color rgba="0.7 0.18 0.0 1.0"/>
-        </material>
-      </visual>
-    </link>
-    <link name="${prefix}link_2">
-      <collision>
-        <geometry>
-          <mesh filename="package://${package_name}/meshes/kr16_r2010_2/collision/link_2_convex.stl"/>
-        </geometry>
-        <origin rpy="-0.0 0.0 -0.0" xyz="0.0 0.0 0.0"/>
-      </collision>
-      <visual>
-        <geometry>
-          <mesh filename="package://${package_name}/meshes/kr16_r2010_2/visual/link_2.stl"/>
-        </geometry>
-        <origin rpy="-0.0 0.0 -0.0" xyz="0.0 0.0 0.0"/>
-        <material name="orange">
-          <color rgba="0.7 0.18 0.0 1.0"/>
-        </material>
-      </visual>
-    </link>
-    <link name="${prefix}link_3">
-      <collision>
-        <geometry>
-          <mesh filename="package://${package_name}/meshes/kr16_r2010_2/collision/link_3_convex.stl"/>
-        </geometry>
-        <origin rpy="-0.0 0.0 -0.0" xyz="0.0 0.0 0.0"/>
-      </collision>
-      <visual>
-        <geometry>
-          <mesh filename="package://${package_name}/meshes/kr16_r2010_2/visual/link_3.stl"/>
-        </geometry>
-        <origin rpy="-0.0 0.0 -0.0" xyz="0.0 0.0 0.0"/>
-        <material name="orange">
-          <color rgba="0.7 0.18 0.0 1.0"/>
-        </material>
-      </visual>
-    </link>
-    <link name="${prefix}link_4">
-      <collision>
-        <geometry>
-          <mesh filename="package://${package_name}/meshes/kr16_r2010_2/collision/link_4_part_1_convex.stl"/>
-        </geometry>
-        <origin rpy="-0.0 0.0 -0.0" xyz="0.0 0.0 0.0"/>
-      </collision>
-      <visual>
-        <geometry>
-          <mesh filename="package://${package_name}/meshes/kr16_r2010_2/visual/link_4.stl"/>
-        </geometry>
-        <origin rpy="-0.0 0.0 -0.0" xyz="0.0 0.0 0.0"/>
-        <material name="orange">
-          <color rgba="0.7 0.18 0.0 1.0"/>
-        </material>
-      </visual>
-    </link>
-    <link name="${prefix}link_4_part_2">
-      <collision>
-        <geometry>
-          <mesh filename="package://${package_name}/meshes/kr16_r2010_2/collision/link_4_convex.stl"/>
-        </geometry>
-        <origin rpy="-0.0 0.0 -0.0" xyz="0.0 0.0 0.0"/>
-      </collision>
-    </link>
-    <link name="${prefix}link_5">
-      <collision>
-        <geometry>
-          <mesh filename="package://${package_name}/meshes/kr16_r2010_2/collision/link_5_convex.stl"/>
-        </geometry>
-        <origin rpy="-0.0 0.0 -0.0" xyz="0.0 0.0 0.0"/>
-      </collision>
-      <visual>
-        <geometry>
-          <mesh filename="package://${package_name}/meshes/kr16_r2010_2/visual/link_5.stl"/>
-        </geometry>
-        <origin rpy="-0.0 0.0 -0.0" xyz="0.0 0.0 0.0"/>
-        <material name="orange">
-          <color rgba="0.7 0.18 0.0 1.0"/>
-        </material>
-      </visual>
-    </link>
-    <link name="${prefix}link_6">
-      <collision>
-        <geometry>
-          <mesh filename="package://${package_name}/meshes/kr16_r2010_2/collision/link_6_convex.stl"/>
-        </geometry>
-        <origin rpy="-0.0 0.0 -0.0" xyz="0.0 0.0 0.0"/>
-      </collision>
-      <visual>
-        <geometry>
-          <mesh filename="package://${package_name}/meshes/kr16_r2010_2/visual/link_6.stl"/>
-        </geometry>
-        <origin rpy="-0.0 0.0 -0.0" xyz="0.0 0.0 0.0"/>
-        <material name="orange">
-          <color rgba="0.7 0.18 0.0 1.0"/>
-        </material>
-      </visual>
-    </link>
-    <xacro:if value="${external_axis}">
-      <joint name="${prefix}parent-rail_base" type="fixed">
-        <parent link="${parent}"/>
-        <child link="${prefix}rail_base"/>
-        <xacro:insert_block name="origin"/>
-      </joint>
-      <joint name="${prefix}linear_rail" type="prismatic">
-        <axis xyz="1 0 0"/>
-        <parent link="${prefix}rail_base"/>
-        <child link="${prefix}rail_carriage"/>
-        <origin rpy="0 0 0" xyz="0 0 0"/>
-        <limit acceleration="0.5" effort="100000.0" lower="-4.5" upper="4.5" velocity="0.175"/>
+      <!-- Origin of the carriage mesh is in an odd location -->
+      <joint name="${prefix}rail_carriage_mesh-rail_carriage" type="fixed">
+        <parent link="${prefix}rail_to_carriage_mount"/>
+        <child link="${prefix}rail_carriage_mesh"/>
+        <xacro:if value="${is_left}">
+          <origin xyz="-0.490 0 0" rpy="0 0 0"/>
+        </xacro:if>
+        <xacro:unless value="${is_left}">
+          <origin xyz="-0.490 0 0" rpy="0 0 0"/>
+        </xacro:unless>
       </joint>
       <joint name="${prefix}base_link" type="fixed">
-        <parent link="${prefix}rail_carriage"/>
+        <parent link="${prefix}rail_to_carriage_mount"/>
         <child link="${prefix}base_link"/>
-        <origin xyz="0 0.159 0" rpy="-1.5708 -1.5708 0"/>
+        <xacro:if value="${is_left}">
+          <origin xyz="0 0.159 0" rpy="-1.5708 -1.5708 0"/>
+        </xacro:if>
+        <xacro:unless value="${is_left}">
+          <origin xyz="0 0.159 0" rpy="-1.5708 -1.5708 0"/>
+        </xacro:unless>
       </joint>
     </xacro:if>
@@ -202,4 +117,114 @@
       </joint>
     </xacro:unless>
+    <link name="${prefix}link_1">
+      <collision>
+        <geometry>
+          <mesh filename="package://${package_name}/meshes/kr16_r2010_2/collision/link_1_convex.stl"/>
+        </geometry>
+        <origin rpy="-0.0 0.0 -0.0" xyz="0.0 0.0 0.0"/>
+      </collision>
+      <visual>
+        <geometry>
+          <mesh filename="package://${package_name}/meshes/kr16_r2010_2/visual/link_1.stl"/>
+        </geometry>
+        <origin rpy="-0.0 0.0 -0.0" xyz="0.0 0.0 0.0"/>
+        <material name="orange">
+          <color rgba="0.7 0.18 0.0 1.0"/>
+        </material>
+      </visual>
+    </link>
+    <link name="${prefix}link_2">
+      <collision>
+        <geometry>
+          <mesh filename="package://${package_name}/meshes/kr16_r2010_2/collision/link_2_convex.stl"/>
+        </geometry>
+        <origin rpy="-0.0 0.0 -0.0" xyz="0.0 0.0 0.0"/>
+      </collision>
+      <visual>
+        <geometry>
+          <mesh filename="package://${package_name}/meshes/kr16_r2010_2/visual/link_2.stl"/>
+        </geometry>
+        <origin rpy="-0.0 0.0 -0.0" xyz="0.0 0.0 0.0"/>
+        <material name="orange">
+          <color rgba="0.7 0.18 0.0 1.0"/>
+        </material>
+      </visual>
+    </link>
+    <link name="${prefix}link_3">
+      <collision>
+        <geometry>
+          <mesh filename="package://${package_name}/meshes/kr16_r2010_2/collision/link_3_convex.stl"/>
+        </geometry>
+        <origin rpy="-0.0 0.0 -0.0" xyz="0.0 0.0 0.0"/>
+      </collision>
+      <visual>
+        <geometry>
+          <mesh filename="package://${package_name}/meshes/kr16_r2010_2/visual/link_3.stl"/>
+        </geometry>
+        <origin rpy="-0.0 0.0 -0.0" xyz="0.0 0.0 0.0"/>
+        <material name="orange">
+          <color rgba="0.7 0.18 0.0 1.0"/>
+        </material>
+      </visual>
+    </link>
+    <link name="${prefix}link_4">
+      <collision>
+        <geometry>
+          <mesh filename="package://${package_name}/meshes/kr16_r2010_2/collision/link_4_part_1_convex.stl"/>
+        </geometry>
+        <origin rpy="-0.0 0.0 -0.0" xyz="0.0 0.0 0.0"/>
+      </collision>
+      <visual>
+        <geometry>
+          <mesh filename="package://${package_name}/meshes/kr16_r2010_2/visual/link_4.stl"/>
+        </geometry>
+        <origin rpy="-0.0 0.0 -0.0" xyz="0.0 0.0 0.0"/>
+        <material name="orange">
+          <color rgba="0.7 0.18 0.0 1.0"/>
+        </material>
+      </visual>
+    </link>
+    <link name="${prefix}link_4_part_2">
+      <collision>
+        <geometry>
+          <mesh filename="package://${package_name}/meshes/kr16_r2010_2/collision/link_4_convex.stl"/>
+        </geometry>
+        <origin rpy="-0.0 0.0 -0.0" xyz="0.0 0.0 0.0"/>
+      </collision>
+    </link>
+    <link name="${prefix}link_5">
+      <collision>
+        <geometry>
+          <mesh filename="package://${package_name}/meshes/kr16_r2010_2/collision/link_5_convex.stl"/>
+        </geometry>
+        <origin rpy="-0.0 0.0 -0.0" xyz="0.0 0.0 0.0"/>
+      </collision>
+      <visual>
+        <geometry>
+          <mesh filename="package://${package_name}/meshes/kr16_r2010_2/visual/link_5.stl"/>
+        </geometry>
+        <origin rpy="-0.0 0.0 -0.0" xyz="0.0 0.0 0.0"/>
+        <material name="orange">
+          <color rgba="0.7 0.18 0.0 1.0"/>
+        </material>
+      </visual>
+    </link>
+    <link name="${prefix}link_6">
+      <collision>
+        <geometry>
+          <mesh filename="package://${package_name}/meshes/kr16_r2010_2/collision/link_6_convex.stl"/>
+        </geometry>
+        <origin rpy="-0.0 0.0 -0.0" xyz="0.0 0.0 0.0"/>
+      </collision>
+      <visual>
+        <geometry>
+          <mesh filename="package://${package_name}/meshes/kr16_r2010_2/visual/link_6.stl"/>
+        </geometry>
+        <origin rpy="-0.0 0.0 -0.0" xyz="0.0 0.0 0.0"/>
+        <material name="orange">
+          <color rgba="0.7 0.18 0.0 1.0"/>
+        </material>
+      </visual>
+    </link>
     <joint name="${prefix}joint_1" type="revolute">
       <axis xyz="0.0 0.0 1.0"/>
