Commit message: feat: add rail_mesh_package override for rail/carriage meshes
Co-Authored-By: Claude Opus 4.8 (1M context) <noreply@anthropic.com>

File: kuka_cybertech_support/urdf/kr16_r2010_2_macro.xacro (robot description, xacro)
@@ -1,5 +1,9 @@
 <?xml version="1.0"?>
 <robot xmlns:xacro="http://wiki.ros.org/xacro">
-  <xacro:macro name="kuka_kr16_r2010_2_robot" params="prefix package_name *origin parent external_axis:=false is_left:=false">
+  <xacro:macro name="kuka_kr16_r2010_2_robot" params="prefix package_name *origin parent external_axis:=false is_left:=false rail_mesh_package:=''">
+    <xacro:property name="rail_mesh_pkg" value="${rail_mesh_package}"/>
+    <xacro:if value="${rail_mesh_pkg == ''}">
+      <xacro:property name="rail_mesh_pkg" value="${package_name}"/>
+    </xacro:if>
     <!-- links - main serial chain -->
     <link name="${prefix}base_link">
@@ -25,5 +29,5 @@
         <visual>
           <geometry>
-            <mesh filename="package://${package_name}/meshes/kr16_r2010_2/visual/rail_base.stl" scale="1 1 1"/>
+            <mesh filename="package://${rail_mesh_pkg}/meshes/kr16_r2010_2/visual/rail_base.stl" scale="1 1 1"/>
           </geometry>
           <material name="grey">
@@ -33,5 +37,5 @@
         <collision>
           <geometry>
-            <mesh filename="package://${package_name}/meshes/kr16_r2010_2/collision/rail_base_convex.stl" scale="1.0 1.1 1.0"/>
+            <mesh filename="package://${rail_mesh_pkg}/meshes/kr16_r2010_2/collision/rail_base_convex.stl" scale="1.0 1.1 1.0"/>
           </geometry>
         </collision>
@@ -67,8 +71,8 @@
           <geometry>
             <xacro:unless value="${is_left}">
-            <mesh filename="package://${package_name}/meshes/kr16_r2010_2/visual/rail_carriage.stl" scale="1 1 1"/>
+            <mesh filename="package://${rail_mesh_pkg}/meshes/kr16_r2010_2/visual/rail_carriage.stl" scale="1 1 1"/>
             </xacro:unless>
             <xacro:if value="${is_left}">
-            <mesh filename="package://${package_name}/meshes/kr16_r2010_2/visual/rail_carriage_mirrored.stl" scale="1 1 1"/>
+            <mesh filename="package://${rail_mesh_pkg}/meshes/kr16_r2010_2/visual/rail_carriage_mirrored.stl" scale="1 1 1"/>
             </xacro:if>
           </geometry>
@@ -80,8 +84,8 @@
           <geometry>
             <xacro:unless value="${is_left}">
-            <mesh filename="package://${package_name}/meshes/kr16_r2010_2/collision/rail_carriage_convex.stl" scale="1.0 1.1 1.0"/>
+            <mesh filename="package://${rail_mesh_pkg}/meshes/kr16_r2010_2/collision/rail_carriage_convex.stl" scale="1.0 1.1 1.0"/>
             </xacro:unless>
             <xacro:if value="${is_left}">
-            <mesh filename="package://${package_name}/meshes/kr16_r2010_2/collision/rail_carriage_convex_mirrored.stl" scale="1.0 1.1 1.0"/>
+            <mesh filename="package://${rail_mesh_pkg}/meshes/kr16_r2010_2/collision/rail_carriage_convex_mirrored.stl" scale="1.0 1.1 1.0"/>
             </xacro:if>
           </geometry>

Commit message: feat: add rail_base_x_offset for per-side rail track alignment
Co-Authored-By: Claude Opus 4.8 (1M context) <noreply@anthropic.com>

File: kuka_cybertech_support/urdf/kr16_r2010_2_macro.xacro (robot description, xacro)
@@ -1,5 +1,5 @@
 <?xml version="1.0"?>
 <robot xmlns:xacro="http://wiki.ros.org/xacro">
-  <xacro:macro name="kuka_kr16_r2010_2_robot" params="prefix package_name *origin parent external_axis:=false is_left:=false rail_mesh_package:=''">
+  <xacro:macro name="kuka_kr16_r2010_2_robot" params="prefix package_name *origin parent external_axis:=false is_left:=false rail_mesh_package:='' rail_base_x_offset:=0">
     <xacro:property name="rail_mesh_pkg" value="${rail_mesh_package}"/>
     <xacro:if value="${rail_mesh_pkg == ''}">
@@ -45,8 +45,8 @@
         <child link="${prefix}rail_base"/>
         <xacro:if value="${is_left}">
-          <origin xyz="0.315 0 0" rpy="3.141592 0 0"/>
+          <origin xyz="${0.315 + rail_base_x_offset} 0 0" rpy="3.141592 0 0"/>
         </xacro:if>
         <xacro:unless value="${is_left}">
-          <origin xyz="${(-4.288 - 0.850 - 4.870 + 0.315)} 0 0" rpy="3.141592 0 0"/>
+          <origin xyz="${(-4.288 - 0.850 - 4.870 + 0.315) + rail_base_x_offset} 0 0" rpy="3.141592 0 0"/>
         </xacro:unless>
       </joint>

Commit message: feat: parameterize base_link mount translation (arm_mount_xyz)
Co-Authored-By: Claude Opus 4.8 (1M context) <noreply@anthropic.com>

File: kuka_cybertech_support/urdf/kr16_r2010_2_macro.xacro (robot description, xacro)
@@ -1,5 +1,5 @@
 <?xml version="1.0"?>
 <robot xmlns:xacro="http://wiki.ros.org/xacro">
-  <xacro:macro name="kuka_kr16_r2010_2_robot" params="prefix package_name *origin parent external_axis:=false is_left:=false rail_mesh_package:='' rail_base_x_offset:=0">
+  <xacro:macro name="kuka_kr16_r2010_2_robot" params="prefix package_name *origin parent external_axis:=false is_left:=false rail_mesh_package:='' rail_base_x_offset:=0 arm_mount_xyz:='0 0.159 0'">
     <xacro:property name="rail_mesh_pkg" value="${rail_mesh_package}"/>
     <xacro:if value="${rail_mesh_pkg == ''}">
@@ -107,8 +107,8 @@
         <child link="${prefix}base_link"/>
         <xacro:if value="${is_left}">
-          <origin xyz="0 0.159 0" rpy="-1.5708 -1.5708 0"/>
+          <origin xyz="${arm_mount_xyz}" rpy="-1.5708 -1.5708 0"/>
         </xacro:if>
         <xacro:unless value="${is_left}">
-          <origin xyz="0 0.159 0" rpy="-1.5708 -1.5708 0"/>
+          <origin xyz="${arm_mount_xyz}" rpy="-1.5708 -1.5708 0"/>
         </xacro:unless>
       </joint>

Commit message: fix(collision): remove errant 10% Y inflation from carriage collision
scale="1.0 1.1 1.0" belongs on the rail body, not the carriage. Applied to the carriage it inflated the collision mesh ~5cm in +Y past the visual, causing spurious link-vs-carriage collisions during dual-arm wash passes.

Co-Authored-By: Claude Opus 4.8 (1M context) <noreply@anthropic.com>

File: kuka_cybertech_support/urdf/kr16_r2010_2_macro.xacro (robot description, xacro)
@@ -84,8 +84,8 @@
           <geometry>
             <xacro:unless value="${is_left}">
-            <mesh filename="package://${rail_mesh_pkg}/meshes/kr16_r2010_2/collision/rail_carriage_convex.stl" scale="1.0 1.1 1.0"/>
+            <mesh filename="package://${rail_mesh_pkg}/meshes/kr16_r2010_2/collision/rail_carriage_convex.stl" scale="1 1 1"/>
             </xacro:unless>
             <xacro:if value="${is_left}">
-            <mesh filename="package://${rail_mesh_pkg}/meshes/kr16_r2010_2/collision/rail_carriage_convex_mirrored.stl" scale="1.0 1.1 1.0"/>
+            <mesh filename="package://${rail_mesh_pkg}/meshes/kr16_r2010_2/collision/rail_carriage_convex_mirrored.stl" scale="1 1 1"/>
             </xacro:if>
           </geometry>

Commit message: Parameterize linear rail position limits
Add rail_lower_limit / rail_upper_limit params (default +-4.5) to the
cybertech linear_rail <limit>, so rail travel range can be set per
consumer (per bay in autowash_config) rather than hardcoded +-4.5.

Co-Authored-By: Claude Opus 4.8 (1M context) <noreply@anthropic.com>

File: kuka_cybertech_support/urdf/kr16_r2010_2_macro.xacro (robot description, xacro)
@@ -1,5 +1,5 @@
 <?xml version="1.0"?>
 <robot xmlns:xacro="http://wiki.ros.org/xacro">
-  <xacro:macro name="kuka_kr16_r2010_2_robot" params="prefix package_name *origin parent external_axis:=false is_left:=false rail_mesh_package:='' rail_base_x_offset:=0 arm_mount_xyz:='0 0.159 0'">
+  <xacro:macro name="kuka_kr16_r2010_2_robot" params="prefix package_name *origin parent external_axis:=false is_left:=false rail_mesh_package:='' rail_base_x_offset:=0 arm_mount_xyz:='0 0.159 0' rail_lower_limit:=-4.5 rail_upper_limit:=4.5">
     <xacro:property name="rail_mesh_pkg" value="${rail_mesh_package}"/>
     <xacro:if value="${rail_mesh_pkg == ''}">
@@ -65,5 +65,5 @@
         <child link="${prefix}rail_to_carriage_mount"/>
         <origin xyz="0 0 0" rpy="3.141592 0 0" />
-        <limit acceleration="0.5" effort="100000.0" lower="-4.5" upper="4.5" velocity="0.175"/>
+        <limit acceleration="0.5" effort="100000.0" lower="${rail_lower_limit}" upper="${rail_upper_limit}" velocity="0.175"/>
       </joint>
       <link name="${prefix}rail_carriage_mesh">

Commit message: Parameterize rail-mesh and carriage transforms via macro params
Replace the hardcoded is_left branches in the parent->rail_base,
rail_carriage_mesh, and base_link joints with macro params:
  - rail_mesh_xyz / rail_mesh_rpy
  - rail_carriage_mesh_xyz / rail_carriage_mesh_rpy
  - carriage_plate_thickness (pure-Y base_link standoff)

Defaults reproduce the previous left-rail values.

Co-Authored-By: Claude Opus 4.8 (1M context) <noreply@anthropic.com>

File: kuka_cybertech_support/urdf/kr16_r2010_2_macro.xacro (robot description, xacro)
@@ -1,5 +1,5 @@
 <?xml version="1.0"?>
 <robot xmlns:xacro="http://wiki.ros.org/xacro">
-  <xacro:macro name="kuka_kr16_r2010_2_robot" params="prefix package_name *origin parent external_axis:=false is_left:=false rail_mesh_package:='' rail_base_x_offset:=0 arm_mount_xyz:='0 0.159 0' rail_lower_limit:=-4.5 rail_upper_limit:=4.5">
+  <xacro:macro name="kuka_kr16_r2010_2_robot" params="prefix package_name *origin parent external_axis:=false is_left:=false rail_mesh_package:='' rail_mesh_xyz:='0 0 0' rail_mesh_rpy:='3.141592 0 0' rail_carriage_mesh_xyz:='-0.490 0 0' rail_carriage_mesh_rpy:='0 0 0' carriage_plate_thickness:=0.159 rail_lower_limit:=-4.5 rail_upper_limit:=4.5">
     <xacro:property name="rail_mesh_pkg" value="${rail_mesh_package}"/>
     <xacro:if value="${rail_mesh_pkg == ''}">
@@ -44,10 +44,5 @@
         <parent link="${parent}"/>
         <child link="${prefix}rail_base"/>
-        <xacro:if value="${is_left}">
-          <origin xyz="${0.315 + rail_base_x_offset} 0 0" rpy="3.141592 0 0"/>
-        </xacro:if>
-        <xacro:unless value="${is_left}">
-          <origin xyz="${(-4.288 - 0.850 - 4.870 + 0.315) + rail_base_x_offset} 0 0" rpy="3.141592 0 0"/>
-        </xacro:unless>
+        <origin xyz="${rail_mesh_xyz}" rpy="${rail_mesh_rpy}"/>
       </joint>
       <!-- The hand measured zero position of the "Kuka mounting pin" relative to the left-most point of the rail -->
@@ -96,20 +91,10 @@
         <parent link="${prefix}rail_to_carriage_mount"/>
         <child link="${prefix}rail_carriage_mesh"/>
-        <xacro:if value="${is_left}">
-          <origin xyz="-0.490 0 0" rpy="0 0 0"/>
-        </xacro:if>
-        <xacro:unless value="${is_left}">
-          <origin xyz="-0.490 0 0" rpy="0 0 0"/>
-        </xacro:unless>
+        <origin xyz="${rail_carriage_mesh_xyz}" rpy="${rail_carriage_mesh_rpy}"/>
       </joint>
       <joint name="${prefix}base_link" type="fixed">
         <parent link="${prefix}rail_to_carriage_mount"/>
         <child link="${prefix}base_link"/>
-        <xacro:if value="${is_left}">
-          <origin xyz="${arm_mount_xyz}" rpy="-1.5708 -1.5708 0"/>
-        </xacro:if>
-        <xacro:unless value="${is_left}">
-          <origin xyz="${arm_mount_xyz}" rpy="-1.5708 -1.5708 0"/>
-        </xacro:unless>
+        <origin xyz="0 ${carriage_plate_thickness} 0" rpy="-1.5708 -1.5708 0"/>
       </joint>
     </xacro:if>

Commit message: feat(cybertech): dull white rail base, black arm base_link
The rail extrusion is painted white on the installed hardware and the KUKA
base casting is black, not orange. Recolour the two visuals to match.

Co-Authored-By: Claude Opus 5 (1M context) <noreply@anthropic.com>

File: kuka_cybertech_support/urdf/kr16_r2010_2_macro.xacro (robot description, xacro)
@@ -19,6 +19,6 @@
         </geometry>
         <origin rpy="-0.0 0.0 -0.0" xyz="0.0 0.0 0.0"/>
-        <material name="orange">
-          <color rgba="0.7 0.18 0.0 1.0"/>
+        <material name="black">
+          <color rgba="0.05 0.05 0.05 1.0"/>
         </material>
       </visual>
@@ -31,6 +31,6 @@
             <mesh filename="package://${rail_mesh_pkg}/meshes/kr16_r2010_2/visual/rail_base.stl" scale="1 1 1"/>
           </geometry>
-          <material name="grey">
-            <color rgba="0.1 0.1 0.1 1.0"/>
+          <material name="rail_white">
+            <color rgba="0.62 0.62 0.60 1.0"/>
           </material>
         </visual>
